File: central-control-unit/central-control-unit/1-wire-bus.sch (KiCad schematic (older format))
At the start: 116 parts, among them P25 1x2_pin_header, P27 1x2_pin_header, P29 1x2_pin_header, P31 1x2_pin_header, P33 1x2_pin_header, P35 1x2_pin_header, P36 1x2_pin_header, P37 1x2_pin_header, P38 1x2_pin_header, P39 1x2_pin_header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

Commit message: Small changes.
Other:
- note added: "Propojka 0R"
Changed lines of the file:
@@
 Wire Wire Line
 	15100 5050 15250 5050
+Text Notes 1650 3950 0    50   ~ 0
+Propojka 0R
 $EndSCHEMATC
