File: central-control-unit/central-control-unit/connectors.sch (KiCad schematic (older format))
At the start: 112 parts, among them J17 1x4_idc_lsa, J18 1x4_idc_lsa, J19 1x4_idc_lsa, J20 1x4_idc_lsa, J21 54601-908WPLF, J22 54601-908WPLF, J23 54601-908WPLF, J24 1x4_idc_lsa, J25 54601-908WPLF, J26 54601-908WPLF, J27 1x4_idc_lsa, J28 1x4_idc_lsa, J29 1x4_idc_lsa, J30 1x4_idc_lsa, J31 1x4_idc_lsa, J32 1x4_idc_lsa, J33 1x4_idc_lsa, J34 1x4_idc_lsa, J35 54601-908WPLF, J36 54601-908WPLF, J37 54601-908WPLF, J38 1x4_idc_lsa, J39 1x4_idc_lsa, J40 1x4_idc_lsa, J41 1x4_idc_lsa, J42 1x4_idc_lsa, J43 54601-908WPLF, J44 54601-908WPLF, J45 1x4_idc_lsa, J46 1x4_idc_lsa, J47 1x3_screw_term_block, J48 1x3_screw_term_block, J49 1x3_screw_term_block, J50 1x3_screw_term_block, J51 1x3_screw_term_block, J52 1x3_screw_term_block, P101 1x3_pin_header, P102 1x3_pin_header, P103 1x3_pin_header, P104 1x3_pin_header, P105 1x3_pin_header, P106 1x3_pin_header, P107 1x3_pin_header, P108 1x3_pin_header, P109 1x3_pin_header, P110 1x3_pin_header, P111 1x3_pin_header, P112 1x3_pin_header, Q50 PMV213SN,215, Q51 PMV213SN,215, Q52 PMV213SN,215, Q53 PMV213SN,215, Q54 PMV213SN,215, Q55 PMV213SN,215, U26 TXS0108E, U27 TLP2345, U28 TLP2345, U29 TLP2345, U30 TLP2345, U31 TLP2345, U32 TLP2345

Commit message: Small changes.
Other:
- note added: "Local thermostat on the first floor."
- note added: "Local thermostat on the ground floor."
- note added: "Zde fyzicky přerušit a napojit na vstup RPI."
Changed lines of the file:
@@
 Wire Wire Line
 	23900 18550 23900 18500
+Text Notes 20900 21400 0    50   ~ 0
+Local thermostat on the ground floor.
+Text Notes 20500 17550 0    50   ~ 0
+Local thermostat on the first floor.
+Text Notes 14650 6550 0    50   ~ 0
+Local thermostat on the ground floor.
+Text Notes 14750 6650 0    50   ~ 0
+Local thermostat on the first floor.
+Text Notes 14450 6350 0    50   ~ 0
+Zde fyzicky přerušit a napojit na vstup RPI.
 $EndSCHEMATC
