File: central-control-unit/central-control-unit/pin-headers.sch (KiCad schematic (older format))
At the start: 5 parts, among them P115 2x20_pin_socket, P116 2x20_pin_header, P4 1x20_pin_socket

Commit message: Small changes.
Other:
- note added: "Local thermostat on the first floor."
- note added: "Local thermostat on the ground floor."
Changed lines of the file:
@@
 Wire Wire Line
 	1300 1400 1300 1700
+Text Notes 5550 1600 0    50   ~ 0
+Local thermostat on the ground floor.
+Text Notes 5500 1450 0    50   ~ 0
+Local thermostat on the first floor.
 $EndSCHEMATC
