File: central-control-unit/central-control-unit/relays-outputs.sch (KiCad schematic (older format))
At the start: 188 parts, among them J10 1x2_screw_term_block, J11 1x2_screw_term_block, J12 AKZ770_3-5.08-V-GREEN, J13 1x2_screw_term_block, J14 1x2_screw_term_block, J15 1x2_screw_term_block, J16 1x2_screw_term_block, J6 1x2_screw_term_block, J7 1x2_screw_term_block, J8 1x2_screw_term_block, J9 1x2_screw_term_block, P10 1x3_pin_header, P11 1x3_pin_header, P12 1x3_pin_header, P13 1x3_pin_header, P14 1x3_pin_header, P15 1x3_pin_header, P16 1x3_pin_header, P17 1x3_pin_header, P18 1x3_pin_header, P19 1x3_pin_header, P20 1x3_pin_header, P21 1x3_pin_header, P22 1x3_pin_header, P23 1x3_pin_header, P24 1x3_pin_header, P5 1x3_pin_header, P6 1x3_pin_header, P7 1x3_pin_header, P8 1x3_pin_header, P9 1x3_pin_header, Q23 AOD458, Q24 AOD458, Q25 AOD458, Q26 AOD458, Q27 AOD458, Q28 AOD458, Q29 PMV213SN,215, Q30 PMV213SN,215, Q31 PMV213SN,215, Q32 PMV213SN,215, Q33 PMV213SN,215, Q34 PMV213SN,215, Q35 AOD458, Q36 AOD458, Q37 AOD458, Q38 AOD458, Q69 PMV213SN,215, Q70 PMV213SN,215, Q71 PMV213SN,215, Q72 PMV213SN,215, Q73 PMV213SN,215, Q74 PMV213SN,215, U13 TLP2345, U14 TLP2345, U15 TLP2345, U16 TLP2345, U17 TLP2345, U18 TLP2345, U19 TLP2345, U20 TLP2345, U21 TLP2345, U22 TLP2345

Commit message: Small changes.
Parts:
- R127, R128, R129, R254, R255, R256, R257, R258, R259: value 4k7 -> 250R
Changed lines of the file:
@@
 P 20750 5100
 F 0 "R127" V 20704 5168 50  0000 L CNN
-F 1 "4k7" V 20795 5168 50  0000 L CNN
+F 1 "250R" V 20795 5168 50  0000 L CNN
 F 2 "resistor_smd_rl:r_1206" H 20750 5100 50  0001 C CNN
 F 3 "" H 20750 5100 50  0001 C CNN
@@
 P 20700 10850
 F 0 "R128" V 20654 10918 50  0000 L CNN
-F 1 "4k7" V 20745 10918 50  0000 L CNN
+F 1 "250R" V 20745 10918 50  0000 L CNN
 F 2 "resistor_smd_rl:r_1206" H 20700 10850 50  0001 C CNN
 F 3 "" H 20700 10850 50  0001 C CNN
@@
 P 20700 16350
 F 0 "R129" V 20654 16418 50  0000 L CNN
-F 1 "4k7" V 20745 16418 50  0000 L CNN
+F 1 "250R" V 20745 16418 50  0000 L CNN
 F 2 "resistor_smd_rl:r_1206" H 20700 16350 50  0001 C CNN
 F 3 "" H 20700 16350 50  0001 C CNN
@@
 P 20750 6900
 F 0 "R259" V 20704 6968 50  0000 L CNN
-F 1 "4k7" V 20795 6968 50  0000 L CNN
+F 1 "250R" V 20795 6968 50  0000 L CNN
 F 2 "resistor_smd_rl:r_1206" H 20750 6900 50  0001 C CNN
 F 3 "" H 20750 6900 50  0001 C CNN
@@
 P 20700 8650
 F 0 "R256" V 20654 8718 50  0000 L CNN
-F 1 "4k7" V 20745 8718 50  0000 L CNN
+F 1 "250R" V 20745 8718 50  0000 L CNN
 F 2 "resistor_smd_rl:r_1206" H 20700 8650 50  0001 C CNN
 F 3 "" H 20700 8650 50  0001 C CNN
@@
 P 20700 12650
 F 0 "R257" V 20654 12718 50  0000 L CNN
-F 1 "4k7" V 20745 12718 50  0000 L CNN
+F 1 "250R" V 20745 12718 50  0000 L CNN
 F 2 "resistor_smd_rl:r_1206" H 20700 12650 50  0001 C CNN
 F 3 "" H 20700 12650 50  0001 C CNN
@@
 P 20700 14400
 F 0 "R258" V 20654 14468 50  0000 L CNN
-F 1 "4k7" V 20745 14468 50  0000 L CNN
+F 1 "250R" V 20745 14468 50  0000 L CNN
 F 2 "resistor_smd_rl:r_1206" H 20700 14400 50  0001 C CNN
 F 3 "" H 20700 14400 50  0001 C CNN
@@
 P 20650 18100
 F 0 "R255" V 20604 18168 50  0000 L CNN
-F 1 "4k7" V 20695 18168 50  0000 L CNN
+F 1 "250R" V 20695 18168 50  0000 L CNN
 F 2 "resistor_smd_rl:r_1206" H 20650 18100 50  0001 C CNN
 F 3 "" H 20650 18100 50  0001 C CNN
@@
 P 20600 19950
 F 0 "R254" V 20554 20018 50  0000 L CNN
-F 1 "4k7" V 20645 20018 50  0000 L CNN
+F 1 "250R" V 20645 20018 50  0000 L CNN
 F 2 "resistor_smd_rl:r_1206" H 20600 19950 50  0001 C CNN
 F 3 "" H 20600 19950 50  0001 C CNN
