File: zone-controller/zone-controller.sch (KiCad schematic (older format))
At the start: 363 parts, among them J1 EBBA-02-C-SS-BU, J10 EBBA-02-C-SS-BU, J11 EBBA-02-C-SS-BU, J12 EBBA-02-C-SS-BU, J13 EBBA-02-C-SS-BU, J14 EBBA-02-C-SS-BU, J15 EBBA-02-C-SS-BU, J16 1x4_idc_lsa, J17 54601-908WPLF, J18 1x4_idc_lsa, J19 EBBA-02-C-SS-BU, J2 EBBA-02-C-SS-BU, J3 EBBA-02-C-SS-BU, J4 EBBA-02-C-SS-BU, J5 EBBA-02-C-SS-BU, J6 EBBA-02-C-SS-BU, J7 EBBA-02-C-SS-BU, J8 EBBA-02-C-SS-BU, J9 EBBA-02-C-SS-BU, P1 1x3_pin_header, P10 1x2_pin_header, P11 1x2_pin_header, P12 1x2_pin_header, P13 1x2_pin_header, P14 1x2_pin_header, P15 1x2_pin_header, P16 1x2_pin_header, P2 1x3_pin_header, P3 1x3_pin_header, P4 1x3_pin_header, P5 1x3_pin_header, P6 1x3_pin_header, P7 1x2_pin_header, P8 1x2_pin_header, P9 1x2_pin_header, Q1 AOD458, Q10 AOD458, Q11 AOD458, Q12 AOD458, Q13 PMV213SN,215, Q14 PMV213SN,215, Q15 AOB1608L, Q17 AOB1608L, Q18 PMV213SN,215, Q19 PMV213SN,215, Q2 AOD458, Q20 AOB1608L, Q21 AOB1608L, Q22 PMV213SN,215, Q23 PMV213SN,215, Q3 AOD458, Q4 AOD458, Q5 AOD458, Q6 AOD458, Q7 AOD458, Q8 AOD458, Q9 AOD458, SW1 SMTS-102-2C2T, SW10 SMTS-102-2C2T, SW11 SMTS-102-2C2T, SW12 SMTS-102-2C2T, SW13 SMTS-102-2C2T, SW2 SMTS-102-2C2T, SW3 SMTS-102-2C2T, SW4 SMTS-102-2C2T, SW5 SMTS-102-2C2T, SW6 SMTS-102-2C2T, SW7 SMTS-102-2C2T, SW8 SMTS-102-2C2T, SW9 SMTS-102-2C2T, U1 TLP2345, U10 TLP2345, U11 TLP2345, U12 TLP2345, U13 TLP2345, U14 TLP2345, U15 TLP2345, U16 TLP2345, U17 TLP2345, U18 TLP2345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

Commit message: Small changes.
Parts:
- removed D47: PMEG40T30EPX, package_sod_rl:sod_128, symbol diode_rl:schottky_diode
- added Q? (x2): 2N7002A-YAN, package_sot_rl:sot_23, symbol unipolar_transistor_rl:n_mosfet_gsd
- added R? (x2): 10k, resistor_smd_rl:r_1206, symbol passive_component_rl:resistor_us
- added R?: 2k2/0.5W, resistor_smd_rl:r_1206, symbol passive_component_rl:resistor_us
- R25: value 7k5 -> 4k7
- R72: value 1k -> 250R
Connections:
- net +24V_A: now also R?.1, R?.1
- net GND_A: now also Q?.2 (S), Q?.2 (S), R?.2
- net LED0_24V: now also Q?.1 (G), R?.1, R?.2; no longer D1.1 (K)
- net PUMP_ACTIVE_0: now also D46.1 (K), R84.2
- new net: D1.1 (K), Q?.3 (D)
- new net: Q?.1 (G), Q?.3 (D), R?.2
Other:
- note added: "Replace the Schottky diode with cable."
- moved on the sheet: C76, D1, D13, D2, J1, Q1, R1, R10, R14, R2, R25, SW1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
