File: zone-controller/the-newest-version/zone-controller.kicad_pcb (KiCad board)
At the start: 2 copper layers, 190 x 153.2 mm, 1103 parts, among them J1 EBBA-02-C-SS-BU, J10 EBBA-02-C-SS-BU, J11 EBBA-02-C-SS-BU, J12 EBBA-02-C-SS-BU, J13 EBBA-02-C-SS-BU, J14 EBBA-02-C-SS-BU, J15 EBBA-02-C-SS-BU, J16 1x4_idc_lsa, J17 54601-908WPLF, J18 1x4_idc_lsa, J19 EBBA-02-C-SS-BU, J2 EBBA-02-C-SS-BU, J3 EBBA-02-C-SS-BU, J4 EBBA-02-C-SS-BU, J5 EBBA-02-C-SS-BU, J6 EBBA-02-C-SS-BU, J7 EBBA-02-C-SS-BU, J8 EBBA-02-C-SS-BU, J9 EBBA-02-C-SS-BU, P1 1x3_pin_header, P10 1x2_pin_header, P11 1x2_pin_header, P12 1x2_pin_header, P13 1x2_pin_header, P14 1x2_pin_header, P15 1x2_pin_header, P16 1x2_pin_header, P2 1x3_pin_header, P3 1x3_pin_header, P4 1x3_pin_header, P5 1x3_pin_header, P6 1x3_pin_header, P7 1x2_pin_header, P8 1x2_pin_header, P9 1x2_pin_header, Q1 AOD458, Q10 AOD458, Q11 AOD458, Q12 AOD458, Q13 PMV213SN,215, Q14 PMV213SN,215, Q15 AOB1608L, Q16 2N7002A-YAN, Q17 AOB1608L, Q18 PMV213SN,215, Q19 PMV213SN,215, Q2 AOD458, Q20 AOB1608L, Q21 AOB1608L, Q22 PMV213SN,215, Q23 PMV213SN,215, Q24 2N7002A-YAN, Q25 2N7002A-YAN, Q26 2N7002A-YAN, Q27 2N7002A-YAN, Q28 2N7002A-YAN, Q29 2N7002A-YAN, Q3 AOD458, Q30 2N7002A-YAN, Q31 2N7002A-YAN, Q32 2N7002A-YAN, Q33 2N7002A-YAN, Q34 2N7002A-YAN, Q35 2N7002A-YAN, Q36 2N7002A-YAN, Q37 2N7002A-YAN, Q38 2N7002A-YAN, Q39 2N7002A-YAN, Q4 AOD458, Q40 2N7002A-YAN, Q41 2N7002A-YAN, Q42 2N7002A-YAN, Q43 2N7002A-YAN, Q44 2N7002A-YAN, Q45 2N7002A-YAN, Q46 2N7002A-YAN, Q5 AOD458, Q6 AOD458, Q7 AOD458, Q8 AOD458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

Commit message: Adding of transistors for LED indication.
Parts:
- added ~: ~, via_pad_rl:via_pad_0.4x0.8, F.Cu at (172.5, 72.6)
- added ~: ~, via_pad_rl:via_pad_0.4x0.8, F.Cu at (151.1, 118.6)
- added ~: ~, via_pad_rl:via_pad_0.4x0.8, F.Cu at (160.5, 128.0)
- added ~: ~, via_pad_rl:via_pad_0.4x0.8, F.Cu at (215.9, 73.2)
- added ~: ~, via_pad_rl:via_pad_0.4x0.8, F.Cu at (215.9, 86.6)
- added ~: ~, via_pad_rl:via_pad_0.4x0.8, F.Cu at (215.9, 97.3)
- added ~: ~, via_pad_rl:via_pad_0.4x0.8, F.Cu at (195.3, 117.9)
- added ~: ~, via_pad_rl:via_pad_0.4x0.8, F.Cu at (169.9, 117.9)
- added ~: ~, via_pad_rl:via_pad_0.4x0.8, F.Cu at (151.1, 128.0)
- added ~: ~, via_pad_rl:via_pad_0.4x0.8, F.Cu at (169.9, 128.0)
- added ~: ~, via_pad_rl:via_pad_0.4x0.8, F.Cu at (148.6, 90.7)
- added ~: ~, via_pad_rl:via_pad_0.4x0.8, F.Cu at (136.9, 99.1)
- added ~: ~, via_pad_rl:via_pad_0.4x0.8, F.Cu at (188.7, 117.9)
- added ~: ~, via_pad_rl:via_pad_0.4x0.8, F.Cu at (160.5, 118.6)
- moved ~ 0.51 mm to (42.4, 33.8)
- moved Q29 0.51 mm to (41.1, 36.3)
- moved ~ 0.25 mm to (123.4, 39.4)
- moved ~ 0.25 mm to (124.7, 14.0)
- moved ~ 0.25 mm to (48.5, 31.2)
Routing:
- net Net-(D1-Pad1): track 5.56 -> 6.64 mm
