File: zone-controller/the-newest-version/zone-controller.sch (KiCad schematic (older format))
At the start: 422 parts, among them J1 EBBA-02-C-SS-BU, J10 EBBA-02-C-SS-BU, J11 EBBA-02-C-SS-BU, J12 EBBA-02-C-SS-BU, J13 EBBA-02-C-SS-BU, J14 EBBA-02-C-SS-BU, J15 EBBA-02-C-SS-BU, J16 1x4_idc_lsa, J17 54601-908WPLF, J18 1x4_idc_lsa, J19 EBBA-02-C-SS-BU, J2 EBBA-02-C-SS-BU, J3 EBBA-02-C-SS-BU, J4 EBBA-02-C-SS-BU, J5 EBBA-02-C-SS-BU, J6 EBBA-02-C-SS-BU, J7 EBBA-02-C-SS-BU, J8 EBBA-02-C-SS-BU, J9 EBBA-02-C-SS-BU, P1 1x3_pin_header, P10 1x2_pin_header, P11 1x2_pin_header, P12 1x2_pin_header, P13 1x2_pin_header, P14 1x2_pin_header, P15 1x2_pin_header, P16 1x2_pin_header, P2 1x3_pin_header, P3 1x3_pin_header, P4 1x3_pin_header, P5 1x3_pin_header, P6 1x3_pin_header, P7 1x2_pin_header, P8 1x2_pin_header, P9 1x2_pin_header, Q1 AOD458, Q10 AOD458, Q11 AOD458, Q12 AOD458, Q13 PMV213SN,215, Q14 PMV213SN,215, Q15 AOB1608L, Q16 2N7002A-YAN, Q17 AOB1608L, Q18 PMV213SN,215, Q19 PMV213SN,215, Q2 AOD458, Q20 AOB1608L, Q21 AOB1608L, Q22 PMV213SN,215, Q23 PMV213SN,215, Q24 2N7002A-YAN, Q25 2N7002A-YAN, Q26 2N7002A-YAN, Q27 2N7002A-YAN, Q28 2N7002A-YAN, Q29 2N7002A-YAN, Q3 AOD458, Q30 2N7002A-YAN, Q31 2N7002A-YAN, Q32 2N7002A-YAN, Q33 2N7002A-YAN, Q34 2N7002A-YAN, Q35 2N7002A-YAN, Q36 2N7002A-YAN, Q37 2N7002A-YAN, Q38 2N7002A-YAN, Q39 2N7002A-YAN, Q4 AOD458, Q40 2N7002A-YAN, Q41 2N7002A-YAN, Q42 2N7002A-YAN, Q43 2N7002A-YAN, Q44 2N7002A-YAN, Q45 2N7002A-YAN, Q46 2N7002A-YAN, Q5 AOD458, Q6 AOD458, Q7 AOD458, Q8 AOD458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

Commit message: Small changes for zone controller.
Parts:
- R127, R129, R130, R131, R135, R136, R139, R140, R141, R142, R143, R144, R145, R146, R147, R148, R151, R152, R157, R158, R159, R160, R161, R162: value 10k -> 24k
- R128, R132, R133, R134, R137, R138, R149, R150, R153, R154, R155, R156: value 2k2/0.5W -> 5k36
- R26, R27, R28, R29, R30, R63, R64, R65, R66, R67, R68: value 7k5 -> 4k7
Other:
- note added: "24 V - 1.55 V (typ.) = 22.45 V\nI = 22.45 / 0.0048 A = 4 677 R"
- note added: "Green LED\n24 V - 3 V (typ.) = 21 V\nI = 21 V / 0.0045 A = 4 666 R"
- note added: "Green LED\n24 V - 3 V (typ.) = 21 V\nI = 21 V / 0.0045 A = 4 666 R\n"
- note added: "Green LED\n5 V - 1.55 V (typ.) = 3.45 V\nI = 3.45 V / 0.005 A = 690 R\n"
- note removed: "24 V - 1.55 V (typ.) = 22.45 V\nI = 22.45 / 0.003 A = 7 483 R"
- note removed: "Green LED\n24 V - 3 V (typ.) = 21 V\nI = 21 V / 0.0045 A = 4 700 R\n"
- note removed: "Green LED\n5 V - 1.55 V (typ.) = 3.45 V\nI = 3 V / 0.005 A = 576 R\n"
