File: central-control-unit/currently-deployed-version/central-control-unit/1-wire-bus.sch (KiCad schematic (older format))
At the start: 116 parts, among them P25 1x2_pin_header, P27 1x2_pin_header, P29 1x2_pin_header, P31 1x2_pin_header, P33 1x2_pin_header, P35 1x2_pin_header, P36 1x2_pin_header, P37 1x2_pin_header, P38 1x2_pin_header, P39 1x2_pin_header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

Commit message: Adding of information about projects.
Other:
- note added: "Jumper 0R"
- note removed: "Propojka 0R"
- moved on the sheet: C60, C61, D41, D42, D43, D44, D45, D46, D47, D48, D49, D50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
