File: central-control-unit/currently-deployed-version/central-control-unit/connectors.sch (KiCad schematic (older format))
At the start: 112 parts, among them J17 1x4_idc_lsa, J18 1x4_idc_lsa, J19 1x4_idc_lsa, J20 1x4_idc_lsa, J21 54601-908WPLF, J22 54601-908WPLF, J23 54601-908WPLF, J24 1x4_idc_lsa, J25 54601-908WPLF, J26 54601-908WPLF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

Commit message: Adding of information about projects.
Other:
- moved on the sheet: C68, C69, C70, C71, C72, C73, C74, C75, C76, C77, C78, C79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
