File: central-control-unit/currently-deployed-version/central-control-unit/i2c-bus.sch (KiCad schematic (older format))
At the start: 113 parts, among them P100 1x2_pin_header, P32 1x2_pin_header, P34 1x2_pin_header, P41 1x2_pin_header, P42 1x2_pin_header, P43 1x2_pin_header, P48 1x2_pin_header, P50 1x2_pin_header, P52 1x2_pin_header, P61 1x2_pin_header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

Commit message: Adding of information about projects.
Other:
- moved on the sheet: C64, C65, C66, C67, D74, D75, D76, D77, D78, D79, D80, D81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
