File: central-control-unit/currently-deployed-version/central-control-unit/logic-or-gates.sch (KiCad schematic (older format))
At the start: 38 parts, among them U10 SN74HCS4075-Q1, U11 SN74HCS4075-Q1, U12 SN74HCS32-Q1, U9 SN74HCS4075-Q1

Commit message: Adding of information about projects.
Other:
- moved on the sheet: C32, C33, C34, C35, C36, C37, C38, C39, R68, R69, R70, R71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
