File: central-control-unit/currently-deployed-version/central-control-unit/pin-headers.sch (KiCad schematic (older format))
At the start: 5 parts, among them P115 2x20_pin_socket, P116 2x20_pin_header, P4 1x20_pin_socket

Commit message: Adding of information about projects.
Other:
- note added: "RPI connection"
- moved on the sheet: P116, P4
