File: central-control-unit/currently-deployed-version/central-control-unit/power-supply.sch (KiCad schematic (older format))
At the start: 141 parts, among them J1 1x2_screw_term_block, J2 1x2_screw_term_block, J3 1x2_screw_term_block, J5 1x2_screw_term_block, Q1 AOB1608L, Q10 PMV213SN,215, Q11 PMV213SN,215, Q12 PMV213SN,215, Q13 PMV213SN,215, Q14 PMV213SN,215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

Commit message: Adding of information about projects.
Other:
- moved on the sheet: C1, C10, C11, C12, C13, C14, C15, C16, C17, C18, C19, C2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
