File: central-control-unit/currently-deployed-version/central-control-unit/relays-outputs.sch (KiCad schematic (older format))
At the start: 188 parts, among them J10 1x2_screw_term_block, J11 1x2_screw_term_block, J12 AKZ770_3-5.08-V-GREEN, J13 1x2_screw_term_block, J14 1x2_screw_term_block, J15 1x2_screw_term_block, J16 1x2_screw_term_block, J6 1x2_screw_term_block, J7 1x2_screw_term_block, J8 1x2_screw_term_block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

Commit message: Adding of information about projects.
Other:
- moved on the sheet: C40, C41, C42, C43, C44, C45, C46, C47, C48, C49, C50, C51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
