File: central-control-unit/currently-deployed-version/switches-with-lcd-display/switches-with-lcd-display.sch (KiCad schematic (older format))
At the start: 76 parts, among them P1 1x20_pin_header, P2 1x3_pin_header, P3 1x3_pin_header, P4 1x3_pin_header, P6 1x3_pin_header, P7 1x16_pin_header, Q1 PMV213SN,215, SW1 SMTS-102-2C2T, SW10 SMTS-102-2C2T, SW2 SMTS-102-2C2T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

Commit message: Change of structure.
Parts:
- R1, R10, R2, R3, R4, R5, R6, R7, R8, R9: value 30R -> 62R
Other:
- note added: "Red LED\n3.3 V - 3 V (typ.) = 0.3 V\nI = 0.3 V / 0.0048 A = 62 R"
- note removed: "Red LED\n3.3 V - 3 V (typ.) = 0.3 V\nI = 0.3 V / 0.01 A = 30 R"
Changed lines of the file:
@@
 	-8650 -5650 -8250 -5650
 Text Notes -7400 -5100 0    50   ~ 0
-Red LED\n3.3 V - 3 V (typ.) = 0.3 V\nI = 0.3 V / 0.01 A = 30 R
+Red LED\n3.3 V - 3 V (typ.) = 0.3 V\nI = 0.3 V / 0.0048 A = 62 R
 $Comp
 L passive_component_rl:resistor_us R2
@@
 AR Path="/69344E39/6948FB55" Ref="R?"  Part="1"
 F 0 "R2" V -7746 -5382 50  0000 L CNN
-F 1 "30R" V -7655 -5382 50  0000 L CNN
+F 1 "62R" V -7655 -5382 50  0000 L CNN
 F 2 "resistor_smd_rl:r_1206" H -7700 -5450 50  0001 C CNN
 F 3 "" H -7700 -5450 50  0001 C CNN
@@
 AR Path="/69344E39/636AD72C" Ref="R?"  Part="1"
 F 0 "R1" V -7846 -2982 50  0000 L CNN
-F 1 "30R" V -7755 -2982 50  0000 L CNN
+F 1 "62R" V -7755 -2982 50  0000 L CNN
 F 2 "resistor_smd_rl:r_1206" H -7800 -3050 50  0001 C CNN
 F 3 "" H -7800 -3050 50  0001 C CNN
@@
 AR Path="/69344E39/636E9CEA" Ref="R?"  Part="1"
 F 0 "R3" V -7946 -1032 50  0000 L CNN
-F 1 "30R" V -7855 -1032 50  0000 L CNN
+F 1 "62R" V -7855 -1032 50  0000 L CNN
 F 2 "resistor_smd_rl:r_1206" H -7900 -1100 50  0001 C CNN
 F 3 "" H -7900 -1100 50  0001 C CNN
@@
 AR Path="/69344E39/6379CCA4" Ref="R?"  Part="1"
 F 0 "R5" V -7696 1468 50  0000 L CNN
-F 1 "30R" V -7605 1468 50  0000 L CNN
+F 1 "62R" V -7605 1468 50  0000 L CNN
 F 2 "resistor_smd_rl:r_1206" H -7650 1400 50  0001 C CNN
 F 3 "" H -7650 1400 50  0001 C CNN
@@
 AR Path="/69344E39/6381D928" Ref="R?"  Part="1"
 F 0 "R6" V -7696 3968 50  0000 L CNN
-F 1 "30R" V -7605 3968 50  0000 L CNN
+F 1 "62R" V -7605 3968 50  0000 L CNN
 F 2 "resistor_smd_rl:r_1206" H -7650 3900 50  0001 C CNN
 F 3 "" H -7650 3900 50  0001 C CNN
@@
 AR Path="/69344E39/6386404E" Ref="R?"  Part="1"
 F 0 "R4" V -7796 6218 50  0000 L CNN
-F 1 "30R" V -7705 6218 50  0000 L CNN
+F 1 "62R" V -7705 6218 50  0000 L CNN
 F 2 "resistor_smd_rl:r_1206" H -7750 6150 50  0001 C CNN
 F 3 "" H -7750 6150 50  0001 C CNN
@@
 AR Path="/69344E39/63B2B9F4" Ref="R?"  Part="1"
 F 0 "R8" V -2446 -932 50  0000 L CNN
-F 1 "30R" V -2355 -932 50  0000 L CNN
+F 1 "62R" V -2355 -932 50  0000 L CNN
 F 2 "resistor_smd_rl:r_1206" H -2400 -1000 50  0001 C CNN
 F 3 "" H -2400 -1000 50  0001 C CNN
@@
 AR Path="/69344E39/63B52F7F" Ref="R?"  Part="1"
 F 0 "R9" V -2396 2768 50  0000 L CNN
-F 1 "30R" V -2305 2768 50  0000 L CNN
+F 1 "62R" V -2305 2768 50  0000 L CNN
 F 2 "resistor_smd_rl:r_1206" H -2350 2700 50  0001 C CNN
 F 3 "" H -2350 2700 50  0001 C CNN
@@
 AR Path="/69344E39/63B8070F" Ref="R?"  Part="1"
 F 0 "R7" V -2546 5568 50  0000 L CNN
-F 1 "30R" V -2455 5568 50  0000 L CNN
+F 1 "62R" V -2455 5568 50  0000 L CNN
 F 2 "resistor_smd_rl:r_1206" H -2500 5500 50  0001 C CNN
 F 3 "" H -2500 5500 50  0001 C CNN
@@
 AR Path="/69344E39/63BAE076" Ref="R?"  Part="1"
 F 0 "R10" V -2346 8718 50  0000 L CNN
-F 1 "30R" V -2255 8718 50  0000 L CNN
+F 1 "62R" V -2255 8718 50  0000 L CNN
 F 2 "resistor_smd_rl:r_1206" H -2300 8650 50  0001 C CNN
 F 3 "" H -2300 8650 50  0001 C CNN
@@
 $EndComp
 $Comp
-L power_rl:PWR_FLAG #FLG?
+L power_rl:PWR_FLAG #FLG0104
 U 1 1 63AE4D86
 P 2550 -2450
-F 0 "#FLG?" H 2550 -2375 50  0001 C CNN
+F 0 "#FLG0104" H 2550 -2375 50  0001 C CNN
 F 1 "PWR_FLAG" H 2550 -2277 50  0000 C CNN
 F 2 "" H 2550 -2450 50  0001 C CNN

Commit message: Adding of information about projects.
Other:
- note added: "Central control unit"
- note added: "For LCD display - controller HD44780"
- note removed: "Potreba uzemnit ramec displeje."
- moved on the sheet: C1, C10, C11, C12, C13, C14, C2, C3, C4, C5, C6, C7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
