File: signalization-by-fireplace/signalization-by-fireplace.sch (KiCad schematic (older format))
At the start: 104 parts, among them J1 2x1x4_idc_lsa, J2 DG301-5.0-3P12, J3 54601-908WPLF, J4 2x1x4_idc_lsa, J5 DG390-5.0-02P-12-00A(H), J6 DG301-5.0-02P-12-00A(H), P1 1x4_pin_socket, P10 1x2_pin_header, P11 1x2_pin_header, P12 1x3_pin_header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

Commit message: Small changes.
Parts:
- C14: value 1,2n -> 1.2nF
Changed lines of the file:
@@
 P 13900 5950
 F 0 "C14" V 13854 6060 50  0000 L CNN
-F 1 "1,2n" V 13945 6060 50  0000 L CNN
+F 1 "1.2nF" V 13945 6060 50  0000 L CNN
 F 2 "capacitor_smd_rl:c_1206" H 13900 5950 50  0001 C CNN
 F 3 "" H 13900 5950 50  0001 C CNN

Commit message: Adding of information about project.
Parts:
- Q1, Q2, Q3, Q4: symbol unipolar_transistor_rl:n_mosfet_gsd -> signalization-by-fireplace-rescue:n_mosfet_gsd-unipolar_transistor_rl
- Q6: symbol unipolar_transistor_rl:p_mosfet -> signalization-by-fireplace-rescue:p_mosfet_gsd-unipolar_transistor_rl
- R24: value 3K16 -> 3k16
Other:
- note added: "1-Wire bus protection"
- note added: "Control LEDs"
- note added: "Differential I2C bus"
- note added: "Input voltage protection"
- note added: "Thermocouple"
- note removed: "54601-908WPLF"
- moved on the sheet: C1, C10, C11, C12, C13, C14, C15, C2, C3, C4, C5, C6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
