File: wall-mounted-room-temperature sensor-ethernet/wall-mounted-room-temperature-sensor-ethernet.sch (KiCad schematic (older format))
At the start: 153 parts, among them J1 rj45, P1 2x3_pins_header, P2 1x9_pin_header, Q1 DMG2307L, Q2 FDC2512, SW1 TVAF18BB, SW2 TVAF18BB, SW3 B3F-4150, SW4 B3F-4150, SW5 B3F-4150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

Commit message: Adding of information about project.
Parts:
- Q1: symbol unipolar_transistor_rl:p_mosfet -> unipolar_transistor_rl:p_mosfet_gsd
Connections:
- net labels added: OTHER_+3V3, SYS_+3V3
- net labels removed: OTHER_+3,3V, SYS_+3,3V
- wire segments 693 -> 692
Other:
- note added: "ESP32-WROVER-IE"
- note added: "Ethernet"
- note added: "Ethernet, LAN Transformer"
- note added: "Menu - buttons"
- note added: "POE - Flyback"
- moved on the sheet: C1, C10, C11, C12, C13, C14, C15, C16, C17, C18, C19, C2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
