File: wall-mounted-room-temperature sensor-wifi/wall-mounted-room-temperature-sensor-wifi.sch (KiCad schematic (older format))
At the start: 50 parts, among them J1 dc_barrel_jack, P1 2x3_pins_header, P2 1x9_pin_header, Q1 DMG2307L, SW1 TVAF18BB, SW2 TVAF18BB, SW3 B3F-4150, SW4 B3F-4150, SW5 B3F-4150, U1 TPS79633KTTR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

Commit message: Adding of information about project.
Other:
- note added: "ESP32-WROVER-IE"
- note added: "Menu - buttons"
- note added: "Power supply"
- moved on the sheet: C1, C10, C11, C12, C13, C14, C15, C16, C2, C3, C4, C5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
