File: zone-controller/currently-deployed-version/zone-controller.sch (KiCad schematic (older format))
At the start: 363 parts, among them J1 EBBA-02-C-SS-BU, J10 EBBA-02-C-SS-BU, J11 EBBA-02-C-SS-BU, J12 EBBA-02-C-SS-BU, J13 EBBA-02-C-SS-BU, J14 EBBA-02-C-SS-BU, J15 EBBA-02-C-SS-BU, J16 1x4_idc_lsa, J17 54601-908WPLF, J18 1x4_idc_lsa, J19 EBBA-02-C-SS-BU, J2 EBBA-02-C-SS-BU, J3 EBBA-02-C-SS-BU, J4 EBBA-02-C-SS-BU, J5 EBBA-02-C-SS-BU, J6 EBBA-02-C-SS-BU, J7 EBBA-02-C-SS-BU, J8 EBBA-02-C-SS-BU, J9 EBBA-02-C-SS-BU, P1 1x3_pin_header, P10 1x2_pin_header, P11 1x2_pin_header, P12 1x2_pin_header, P13 1x2_pin_header, P14 1x2_pin_header, P15 1x2_pin_header, P16 1x2_pin_header, P2 1x3_pin_header, P3 1x3_pin_header, P4 1x3_pin_header, P5 1x3_pin_header, P6 1x3_pin_header, P7 1x2_pin_header, P8 1x2_pin_header, P9 1x2_pin_header, Q1 AOD458, Q10 AOD458, Q11 AOD458, Q12 AOD458, Q13 PMV213SN,215, Q14 PMV213SN,215, Q15 AOB1608L, Q17 AOB1608L, Q18 PMV213SN,215, Q19 PMV213SN,215, Q2 AOD458, Q20 AOB1608L, Q21 AOB1608L, Q22 PMV213SN,215, Q23 PMV213SN,215, Q3 AOD458, Q4 AOD458, Q5 AOD458, Q6 AOD458, Q7 AOD458, Q8 AOD458, Q9 AOD458, SW1 SMTS-102-2C2T, SW10 SMTS-102-2C2T, SW11 SMTS-102-2C2T, SW12 SMTS-102-2C2T, SW13 SMTS-102-2C2T, SW2 SMTS-102-2C2T, SW3 SMTS-102-2C2T, SW4 SMTS-102-2C2T, SW5 SMTS-102-2C2T, SW6 SMTS-102-2C2T, SW7 SMTS-102-2C2T, SW8 SMTS-102-2C2T, SW9 SMTS-102-2C2T, U1 TLP2345, U10 TLP2345, U11 TLP2345, U12 TLP2345, U13 TLP2345, U14 TLP2345, U15 TLP2345, U16 TLP2345, U17 TLP2345, U18 TLP2345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

Commit message: Change of structure.
Parts:
- R72: value 1k -> 250R
Changed lines of the file:
@@
 P 5050 12850
 F 0 "R72" V 5004 12918 50  0000 L CNN
-F 1 "1k" V 5095 12918 50  0000 L CNN
+F 1 "250R" V 5095 12918 50  0000 L CNN
 F 2 "resistor_smd_rl:r_1206" H 5050 12850 50  0001 C CNN
 F 3 "" H 5050 12850 50  0001 C CNN

Commit message: Split project to sheets and adding of description about project.
Parts:
- removed C1, C12, C13, C14, C18, C19, C2, C20, C24, C25, C26, C3, C30, C31, C32, C36, C37, C38, C42, C43, C44, C48, C49, C50, C67, C68, C71, C72, C73, C74, C75, C76, C77, C78, C79, C80, C81, C82: 100nF, capacitor_smd_rl:c_1206, symbol passive_component_rl:capacitor
- removed C10: 1.2nF, capacitor_smd_rl:c_1206, symbol passive_component_rl:capacitor
- removed C11, C15, C16, C17, C21, C22, C23, C27, C28, C29, C33, C34, C35, C39, C4, C40, C41, C45, C46, C47, C5, C51, C52, C53, C6, C66, C7, C70: 1uF, capacitor_smd_rl:c_1206, symbol passive_component_rl:capacitor
- removed C54, C58, C63, C69: 10uF, capacitor_smd_rl:c_1206, symbol passive_component_rl:capacitor
- removed C55, C64: 1000pF, capacitor_smd_rl:c_1206, symbol passive_component_rl:capacitor
- removed C56, C65: 33nF, capacitor_smd_rl:c_1206, symbol passive_component_rl:capacitor
- removed D1, D10, D11, D12, D26, D27, D28, D29, D30, D31, D8, D9: LL-504PGC1E-G5-2B, led_tht_rl:led_d5mm_2.54mm, symbol diode_rl:LED
- removed D13, D14, D15, D16, D18, D19, D32, D33, D34, D35, D36, D37: SMCJ24A-CD, diode_smd_rl:smc, symbol diode_rl:undir_transil
- removed D17, D45, D54: LL-503VC1E-4C, led_tht_rl:led_d5mm_2.54mm, symbol diode_rl:LED
- removed D2, D20, D21, D22, D23, D24, D25, D3, D4, D5, D6, D7: STPS160A, diode_smd_rl:sma, symbol diode_rl:schottky_diode
- removed D39, D48: SMBJ24CA-TR, diode_smd_rl:smb, symbol diode_rl:bidir_transil
- removed D40, D41, D49, D51: BAV20WS-DC, package_sod_rl:sod_323, symbol diode_rl:rectifier_diode
- removed D43, D53: TZMB27-GS08, package_sod_rl:minimelf_sod_80, symbol diode_rl:zener_diode
- removed D47: PMEG40T30EPX, package_sod_rl:sod_128, symbol diode_rl:schottky_diode
- removed D50: SMCJ5.0CA-13-F, diode_smd_rl:smc, symbol diode_rl:bidir_transil
- removed D52: SMDA05CDR2G, package_soic_rl:soic_8_3.9mmx4.9mm, symbol diode_rl:SMDA05CDR2G
- removed J1, J10, J11, J12, J13, J14, J2, J3, J4, J5, J6, J7, J8, J9: EBBA-02-C-SS-BU, terminal_block_tht_rl:EBBA-02-C-SS-BU, symbol connector_rl:1x2_screw_term_block
- removed J16, J18: 1x4_idc_lsa, connector_rl:1x4_idc_lsa_connector_general, symbol connector_rl:1x4_idc_lsa
- removed J17: 54601-908WPLF, connector_rl:rj45_54601-908WPLF, symbol connector_rl:rj45
- removed P10, P11, P12, P13, P14, P15, P16, P7, P8, P9: 1x2_pin_header, connector_smd_pinheader_2.54mm_rl:1x2_pinheader_2.54mm_vertical, symbol connector_rl:1x2_pin_header
- removed Q1, Q10, Q11, Q12, Q2, Q3, Q4, Q5, Q6, Q7, Q8, Q9: AOD458, package_to_rl:to_252_2, symbol unipolar_transistor_rl:n_mosfet_gsd
- removed Q15, Q17, Q20, Q21: AOB1608L, package_to_rl:to_263_2, symbol unipolar_transistor_rl:n_mosfet_gsd
- removed Q18, Q19, Q22, Q23: PMV213SN,215, package_sot_rl:sot_23, symbol unipolar_transistor_rl:n_mosfet_gsd
- removed R1, R102, R20, R21, R22, R23, R24, R57, R58, R59, R60, R61, R62, R83: 2k2/0.5W, resistor_smd_rl:r_1206, symbol passive_component_rl:resistor_us
- removed R10, R11, R12, R13, R37, R38, R39, R40, R41, R42, R8, R9: NC (10k), resistor_smd_rl:r_1206, symbol passive_component_rl:resistor_us
- removed R100, R101: 4k7, resistor_smd_rl:r_1206, symbol passive_component_rl:resistor_us
- removed R117, R121, R122, R126: 210R, resistor_smd_rl:r_1206, symbol passive_component_rl:resistor_us
- removed R118, R120, R123, R125: 390R, resistor_smd_rl:r_1206, symbol passive_component_rl:resistor_us
- removed R119, R124: 100R/120R, resistor_smd_rl:r_1206, symbol passive_component_rl:resistor_us
- removed R14, R15, R16, R17, R18, R19, R43, R44, R53, R54, R55, R56: 1k, resistor_smd_rl:r_1206, symbol passive_component_rl:resistor_us
- removed R2, R3, R31, R32, R33, R34, R35, R36, R4, R5, R6, R7: 1k15, resistor_smd_rl:r_1206, symbol passive_component_rl:resistor_us
- removed R25, R26, R27, R28, R29, R30, R63, R64, R65, R66, R67, R68: 7k5, resistor_smd_rl:r_1206, symbol passive_component_rl:resistor_us
- removed R46, R81, R82, R98, R99: 100k, resistor_smd_rl:r_1206, symbol passive_component_rl:resistor_us
- removed R47: 3k16, resistor_smd_rl:r_1206, symbol passive_component_rl:resistor_us
- removed R48: 30k, resistor_smd_rl:r_1206, symbol passive_component_rl:resistor_us
- removed R49: 200R, resistor_smd_rl:r_1206, symbol passive_component_rl:resistor_us
- removed R50: 200k, trimmer_tht_rl:trimmer_t93yb, symbol passive_component_rl:resistor_variable_us
- removed R51: 5k36, resistor_smd_rl:r_1206, symbol passive_component_rl:resistor_us
- removed R52: 604R, resistor_smd_rl:r_1206, symbol passive_component_rl:resistor_us
- removed R70, R87: 24k, resistor_smd_rl:r_1206, symbol passive_component_rl:resistor_us
- removed R71, R88: 2k67, resistor_smd_rl:r_1206, symbol passive_component_rl:resistor_us
- removed R73, R89: 47k5, resistor_smd_rl:r_1206, symbol passive_component_rl:resistor_us
- removed R74, R90: 9k76, resistor_smd_rl:r_1206, symbol passive_component_rl:resistor_us
- removed R75, R91: 25m, resistor_smd_rl:r_1206, symbol passive_component_rl:resistor_us
- removed R76, R92: 1M, resistor_smd_rl:r_1206, symbol passive_component_rl:resistor_us
- removed R78, R93: 14k3, resistor_smd_rl:r_1206, symbol passive_component_rl:resistor_us
- removed R94, R95, R96, R97: 10R/0.5W, resistor_smd_rl:r_1206, symbol passive_component_rl:resistor_us
- removed SW1, SW10, SW11, SW12, SW2, SW3, SW4, SW5, SW6, SW7, SW8, SW9: SMTS-102-2C2T, switch_tht_rl:SMTS-102-2C2T, symbol switch_rl:SMTS-102-2C2T
- removed U1, U10, U11, U12, U13, U14, U15, U16, U17, U18, U19, U2, U20, U21, U22, U23, U24, U25, U26, U5, U6, U7, U8, U9: TLP2345, package_so_rl:so_6, symbol optocoupler_rl:TLP2345
- removed U27, U30: LM5069, package_vssop_rl:vssop_10, symbol power_management_rl:LM5069
- removed U31: PCA9615, package_tssop_rl:tssop_10, symbol interface_i2c_rl:PCA9615
- removed U4: TPS26600, package_htssop_rl:htssop_16_6.6mm×5.1mm, symbol power_management_rl:TPS26600
Connections:
- net PUMP_ACTIVE_0: now also D46.1 (K), R84.2
- no-connect marks 16 -> 4
Other:
- note added: "Controller for valve outputs."
- note added: "Green LED\n5 V - 1.55 V (typ.) = 3.45 V\nI = 3.45 V / 0.005 A = 690 R\n"
- note added: "Manual switch for pump."
- note added: "PE"
- note added: "Signal output for a pump."
- note removed: "24 V - 1.55 V (typ.) = 22.45 V\nI = 22.45 / 0.003 A = 7 483 R"
- note removed: "27 V"
- note removed: "390R-100R-390R\n600R-120R-600R"
- note removed: "5 V - 1.55 V (typ.) = 3.45 V\nI = 3,45 V / 0.003 A = 1 150 R"
- note removed: "5 V - 1.55 V (typ.) = 3.45 V\nI = 3.45 V / 0.003 A = 1 150 R"
- note removed: "Fault: log. 0"
- note removed: "Green LED\n24 V - 3 V (typ.) = 21 V\nI = 21 V / 0.00954 A = 2 200 R\n"
- note removed: "Green LED\n5 V - 1.55 V (typ.) = 3.45 V\nI = 3 V / 0.01 A = 345 R\n"
- note removed: "I=0,073 A (0,13 A) => max. current\n120k - 5k36 = 114,64k"
- note removed: "Ilimit(nominal) = 2.2 A\nIlimit(min) = 1.94 A\nIlimit(max) = 2.46 A"
- note removed: "Input\nvoltage \n+24 V"
- note removed: "Input\nvoltage \n+5 V"
- note removed: "Max. 4.72 W"
- note removed: "Output voltage +5 V"
- note removed: "Overvoltage 5,25 V\nUndervoltage 4,75"
- note removed: "Red LED\n24 V - 2 V (typ.) = 22 V\nI = 22 V / 0.01 A = 2200R\n"
- note removed: "Red LED\n5 V - 2 V (typ.) = 3 V\nI = 3 V / 0.005 A = 600 R\n"
- note removed: "Timer: 1.55 ms"
- note removed: "Uuvh = 15.6 V\nUuvl = 14.6 V\n\nUovh = 25 V\nUovl = 24.5 V"
- moved on the sheet: C57, C59, C60, C61, C62, C8, C9, D38, D42, D44, D46, J15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
