File: kicad-v7.0.9/zone-controller/v10.0_v2.0_reference/outputs-switches-6-11.kicad_sch (KiCad schematic)
At the start: 84 parts, among them J10 EBBA-02-C-SS-BU, J11 EBBA-02-C-SS-BU, J12 EBBA-02-C-SS-BU, J7 EBBA-02-C-SS-BU, J8 EBBA-02-C-SS-BU, J9 EBBA-02-C-SS-BU, Q10 AOD458, Q11 AOD458, Q12 AOD458, Q35 2N7002A-YAN, Q36 2N7002A-YAN, Q37 2N7002A-YAN, Q38 2N7002A-YAN, Q39 2N7002A-YAN, Q40 2N7002A-YAN, Q41 2N7002A-YAN, Q42 2N7002A-YAN, Q43 2N7002A-YAN, Q44 2N7002A-YAN, Q45 2N7002A-YAN, Q46 2N7002A-YAN, Q7 AOD458, Q8 AOD458, Q9 AOD458, SW10 SMTS-102-2C2T, SW11 SMTS-102-2C2T, SW12 SMTS-102-2C2T, SW7 SMTS-102-2C2T, SW8 SMTS-102-2C2T, SW9 SMTS-102-2C2T

Commit message: Zone controller. Change library. Small changes in schematic a PCB.
Parts:
- C77, C78, C79, C80, C81, C82: symbol passive_component_rl:capacitor -> capacitor_smd_rl:c_1206
- D20, D21, D22, D23, D24, D25: symbol diode_rl:schottky_diode -> diode_smd_rl:STPS160A
- D26, D27, D28, D29, D30, D31: symbol diode_rl:LED -> led_tht_rl:LL-504PGC1E-G5-2B
- J10, J11, J12, J7, J8, J9: symbol connector_rl:1x2_screw_term_block -> terminal_block_tht_rl:EBBA-02-C-SS-BU
- Q10, Q11, Q12, Q7, Q8, Q9: symbol unipolar_transistor_rl:n_mosfet_gsd -> unipolar_transistor_smd_rl:AOD458
- Q35, Q36, Q37, Q38, Q39, Q40, Q41, Q42, Q43, Q44, Q45, Q46: symbol unipolar_transistor_rl:n_mosfet_gsd -> unipolar_transistor_smd_rl:2N7002A-YAN
- R145, R146, R147, R148, R149, R150, R151, R152, R153, R154, R155, R156, R157, R158, R159, R160, R161, R162, R37, R38, R39, R40, R41, R42, R43, R44, R53, R54, R55, R56, R57, R58, R59, R60, R61, R62: symbol passive_component_rl:resistor_us -> resistor_smd_rl:r_1206_us
- SW10, SW11, SW12, SW7, SW8, SW9: symbol switch_rl:SMTS-102-2C2T -> switch_tht_rl:SMTS-102-2C2T
Other:
- moved on the sheet: D20, D21, D22, D23, D24, D25
