File: kicad-v7.0.9/wall-mounted-room-temperature sensor-wifi/v4/wall-mounted-room-temperature-sensor-wifi.kicad_pcb (KiCad board)
At the start: 2 copper layers, 107 x 90 mm, 52 parts, among them J1 dc_barrel_jack, P1 2x3_pins_header, P2 1x9_pinsocket, Q1 DMG2307L, SW1 TVAF18BB, SW2 TVAF18BB, SW3 B3F-4150, SW4 B3F-4150, SW5 B3F-4150, U1 TPS79633KTTR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

Commit message: Wall mounted room temperature sensor - WiFi. Small changes in schematic a PCB.
Parts:
- removed ~ (x2): mounting_hole_3.2mm_5.5mm, mounting_hole_rl:mounting_hole_3.2mm_5.5mm
- added H1: mounting_hole_2.2x4.4mm, mounting_hole_rl:mounting_hole_2.2x4.4mm, F.Cu at (41.3, 80.0)
- added H10: mounting_hole_3.2x5.5mm, mounting_hole_rl:mounting_hole_3.2x5.5mm, F.Cu at (61.0, 91.7)
- added H11: mounting_hole_3.2x5.5mm, mounting_hole_rl:mounting_hole_3.2x5.5mm, F.Cu at (61.0, 125.7)
- added H2: mounting_hole_2.2x4.4mm, mounting_hole_rl:mounting_hole_2.2x4.4mm, F.Cu at (105.4, 85.7)
- added H3: mounting_hole_2.2x4.4mm, mounting_hole_rl:mounting_hole_2.2x4.4mm, F.Cu at (64.1, 99.7)
- added H4: mounting_hole_2.2x4.4mm, mounting_hole_rl:mounting_hole_2.2x4.4mm, F.Cu at (141.6, 110.5)
- added H5: mounting_hole_2.2x4.4mm, mounting_hole_rl:mounting_hole_2.2x4.4mm, F.Cu at (83.2, 123.8)
- added H6: mounting_hole_2.2x4.4mm, mounting_hole_rl:mounting_hole_2.2x4.4mm, F.Cu at (41.9, 134.6)
- added H7: mounting_hole_2.2x4.4mm, mounting_hole_rl:mounting_hole_2.2x4.4mm, F.Cu at (83.2, 146.1)
- added H8: mounting_hole_2.2x4.4mm, mounting_hole_rl:mounting_hole_2.2x4.4mm, F.Cu at (59.1, 155.6)
- added H9: mounting_hole_2.2x4.4mm, mounting_hole_rl:mounting_hole_2.2x4.4mm, F.Cu at (141.6, 155.6)
- J1: value dc_barrel_jack -> PC-GK2.1; footprint dc_barrel_jack_rl:PC-GK2.1 -> dc_barrel_jack_tht_rl:PC-GK2.1
- P1: value 2x3_pins_header -> 2x3_MLW06A
- P2: value 1x9_pinsocket -> DS1023-1-9S21
Routing:
- net GND: vias 45 -> 46
Other:
- outline, holes or cut-outs redrawn
