File: kicad-v7.0.9/wall-mounted-room-temperature sensor-ethernet/v2.0/wall-mounted-room-temperature-sensor-ethernet.kicad_sch (KiCad schematic)
At the start: 153 parts, among them J1 rj45, P1 2x3_MLW06A, P2 1x9_pin_socket, Q1 DMG2307L, Q2 FDC2512, SW1 TVAF18BB, SW2 TVAF18BB, SW3 B3F-4150, SW4 B3F-4150, SW5 B3F-4150, T1 SM13126PEL, T2 POE70P-50L, U1 TPS79633KTTR, U2 TPS7A8033DRBR, U3 W5500, U4 TPS23753A, U5 FOD817AS, U6 ESP32-WROVER-IE, U7 DS18B20, Y1 ABLS2-25.000MHZ-D4YF-T - 25MHz

Commit message: Wall mounted room temperature sensor - ethernet. Change library. Small changes in schematic a PCB.
Parts:
- added H1, H10, H2, H3, H4, H5, H6, H7, H8, H9: mounting_hole_2.2x4.4mm, mounting_hole_rl:mounting_hole_2.2x4.4mm, symbol mounting_hole_rl:mounting_hole_2.2x4.4mm
- added H11, H12: mounting_hole_3.2x5.5mm, mounting_hole_rl:mounting_hole_3.2x5.5mm, symbol mounting_hole_rl:mounting_hole_3.2x5.5mm
- C1, C10, C11, C12, C13, C14, C15, C16, C17, C18, C19, C2, C20, C22, C24, C25, C26, C29, C3, C30, C31, C32, C33, C34, C35, C37, C38, C39, C4, C40, C42, C43, C44, C45, C46, C49, C5, C50, C51, C52, C53, C54, C55, C56, C57, C58, C6, C7, C8, C9: symbol passive_component_rl:capacitor -> capacitor_smd_rl:c_0805
- C21, C27, C36: symbol passive_component_rl:capacitor -> capacitor_smd_rl:c_1206
- C23: footprint elec_capacitor_smd_rl:elec_c_6.3x7.7 -> capacitor_elec_smd_rl:c_elec_6.3x7.7; symbol passive_component_rl:capacitor_elec -> capacitor_elec_smd_rl:c_elec_6.3x7.7
- C28, C47: footprint elec_capacitor_smd_rl:elec_c_4x5.8 -> capacitor_elec_smd_rl:c_elec_4x5.8; symbol passive_component_rl:capacitor_elec -> capacitor_elec_smd_rl:c_elec_4x5.8
- C41, C48: footprint capacitor_smd_rl:c_1812_gal_space -> capacitor_smd_rl:c_1812; symbol passive_component_rl:capacitor -> capacitor_smd_rl:c_1812
- D1, D2: symbol bridge_rectifier_rl:HD01-T -> bridge_rectifier_smd_rl:HD01-T
- D10: symbol diode_rl:schottky_diode -> diode_smd_rl:SSC54-E3/57T
- D11, D12, D16, D17, D18, D19, D20: symbol diode_rl:undir_transil -> transil_diode_smd_rl:SD05.TCT
- D13, D14, D15, D5: symbol wall-mounted-room-temperature-sensor-ethernet-rescue:PUSB3AB4-diode_rl -> transil_diode_smd_rl:PHDMI2AB4Z
- D21: symbol diode_rl:DS9503_us -> transil_diode_smd_rl:DS9503_us
- D3: symbol diode_rl:schottky_diode -> diode_smd_rl:BAT60B
- D4: symbol diode_rl:undir_transil -> transil_diode_smd_rl:SMAJ58A
- D6: symbol diode_rl:rectifier_diode -> diode_smd_rl:BAV16W-7
- D7: symbol diode_rl:rectifier_diode -> diode_smd_rl:MURA120
- D8: symbol diode_rl:BAV99 -> diode_smd_rl:BAV99
- D9: symbol reference_voltage_rl:TLV431ACDBZR -> reference_voltage_smd_rl:TLV431ACDBZR
- GDT1: symbol gas_discharge_tube_rl:2051-09-SM-RPLF -> gas_discharge_tube_smd_rl:2051-09-SM-RPLF
- J1: value rj45 -> 54601-908WPLF; symbol connector_rl:rj45 -> connector_rj45_tht_rl:54601-908WPLF
- JP1, JP2, JP3: value solder_jumper_2_open -> solder_jumper_2_open_rect_1x1.5mm; footprint solder_jumper_rl:solder_jumper_2_open_rect_1x1,5mm -> solder_jumper_rl:solder_jumper_2_open_rect_1x1.5mm; symbol solder_jumper_rl:solder_jumper_2_open -> solder_jumper_rl:solder_jumper_2_open_rect_1x1.5mm; now left out of the parts list
- L1, L2: footprint resistor_smd_rl:r_0805 -> inductor_smd_rl:ferrite_bead_0805; symbol passive_component_rl:inductor -> ferrite_bead_smd_rl:MMZ2012R150A
- L3: footprint resistor_smd_rl:r_0805 -> inductor_smd_rl:ferrite_bead_0805; symbol passive_component_rl:inductor -> ferrite_bead_smd_rl:BLM21PG121SN1D
- L4: value 4,7uH/1,5A -> DO1608C-472ML; symbol passive_component_rl:inductor -> inductor_smd_rl:DO1608C-472ML
- P2: value 1x9_pin_socket -> DS1023-1-9S21; symbol connector_rl:1x9_pin_socket -> connector_tht_pin_socket_2.54mm_rl:DS1023-1-9S21
- Q1: symbol unipolar_transistor_rl:p_mosfet_gsd -> unipolar_transistor_smd_rl:DMG2307L
- Q2: symbol unipolar_transistor_rl:FDC2512 -> unipolar_transistor_smd_rl:FDC2512
- R1, R11, R13, R14, R15, R16, R17, R18, R19, R2, R20, R21, R22, R23, R24, R25, R26, R27, R28, R29, R3, R31, R32, R34, R35, R36, R37, R38, R39, R4, R40, R41, R42, R43, R44, R45, R46, R5, R6, R7, R8, R9: symbol passive_component_rl:resistor_us -> resistor_smd_rl:r_0805_us
- R10, R12, R30, R33: symbol passive_component_rl:resistor_us -> resistor_smd_rl:r_1206_us
- SW1, SW2: symbol microswitch_rl:TVAF18BB -> microswitch_smd_rl:TVAF18BB
- SW3, SW4, SW5: symbol microswitch_rl:B3F-4150 -> microswitch_tht_rl:B3F-4150
- T1: symbol transformer_rl:SM13126PEL -> transformer_smd_rl:SM13126PEL
- T2: symbol bound_inductor_rl:POE70P-50L -> bound_inductor_smd_rl:POE70P-50L
- U5: symbol optocoupler_rl:FOD817AS -> optocoupler_smd_rl:FOD817AS
- Y1: symbol Device:Crystal -> crystal_smd_rl:ABLS2-25.000MHZ-D4YF-T
Other:
- note added: "4.7uH/1.5A"
- note added: "Mounting hole for screws"
- note added: "Mounting holes"
- note removed: "DO1608C-472ML"
- moved on the sheet: D10, D3, D6, D7
