File: kicad-v7.0.9/testing-board/v1.0_v1.0/testing-board.kicad_pcb (KiCad board)
At the start: 2 copper layers, 31.1 x 73 mm, 39 parts, among them J1 54601-908WPLF, J2 1x2_screw_term_block, P1 1x3_pin_header, P10 1x2_pin_header, P11 1x2_pin_header, P12 1x2_pin_header, P13 1x2_pin_header, P14 1x2_pin_header, P2 1x3_pin_socket, P3 1x4_pin_header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

Commit message: Testing board. Change library. Small changes in schematic a PCB.
Parts:
- removed ~ (x2): pad_3x5mm, pad_rl:pad_3x5mm
- added H1: mounting_hole_pad_3.2x5mm, mounting_hole_pad_rl:mounting_hole_pad_3.2x5mm, F.Cu at (118.7, 65.4)
- added H2: mounting_hole_pad_3.2x5mm, mounting_hole_pad_rl:mounting_hole_pad_3.2x5mm, F.Cu at (118.7, 106.0)
- J2: value 1x2_screw_term_block -> EBBA-02-C-SS-BU
- P1: value 1x3_pin_header -> DS1021-1-3SF11-B
- P10, P11, P12, P13, P14, P5, P6, P7, P8, P9: value 1x2_pin_header -> 10129380-902001BLF
- P2: value 1x3_pin_socket -> DS1023-1-3S21
- P3: value 1x4_pin_header -> DS1021-1-4SF11-B
- P4: value 1x4_pin_socket -> DS1023-1-4S21
