File: kicad-v7.0.9/testing-board/v1.0_v1.0/testing-board.kicad_sch (KiCad schematic)
At the start: 37 parts, among them J1 54601-908WPLF, J2 1x2_screw_term_block, P1 1x3_pin_header, P10 1x2_pin_header, P11 1x2_pin_header, P12 1x2_pin_header, P13 1x2_pin_header, P14 1x2_pin_header, P2 1x3_pin_socket, P3 1x4_pin_header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

Commit message: Testing board. Change library. Small changes in schematic a PCB.
Parts:
- added H1, H2: mounting_hole_pad_3.2x5mm, mounting_hole_pad_rl:mounting_hole_pad_3.2x5mm, symbol mounting_hole_pad_rl:mounting_hole_pad_3.2x5mm
- C1, C2, C3, C4: symbol passive_component_rl:capacitor -> capacitor_smd_rl:c_1206
- J1: symbol connector_rl:rj45 -> connector_rj45_tht_rl:54601-908WPLF
- J2: value 1x2_screw_term_block -> EBBA-02-C-SS-BU; symbol connector_rl:1x2_screw_term_block -> terminal_block_tht_rl:EBBA-02-C-SS-BU
- P1: value 1x3_pin_header -> DS1021-1-3SF11-B; symbol connector_rl:1x3_pin_header -> connector_tht_pin_header_2.54mm_rl:DS1021-1-3SF11-B
- P10, P11, P12, P13, P14, P5, P6, P7, P8, P9: value 1x2_pin_header -> 10129380-902001BLF; symbol connector_rl:1x2_pin_header -> connector_smd_pin_header_2.54mm_rl:10129380-902001BLF
- P2: value 1x3_pin_socket -> DS1023-1-3S21; symbol connector_rl:1x3_pin_socket -> connector_tht_pin_socket_2.54mm_rl:DS1023-1-3S21
- P3: value 1x4_pin_header -> DS1021-1-4SF11-B; symbol connector_rl:1x4_pin_header -> connector_tht_pin_header_2.54mm_rl:DS1021-1-4SF11-B
- P4: value 1x4_pin_socket -> DS1023-1-4S21; symbol connector_rl:1x4_pin_socket -> connector_tht_pin_socket_2.54mm_rl:DS1023-1-4S21
- R1, R10, R11, R12, R13, R14, R15, R16, R2, R3, R4, R5, R6, R7, R8, R9: symbol passive_component_rl:resistor_us -> resistor_smd_rl:r_1206_us
- U1: Manufacturer (none) -> NXP Semiconductors
Connections:
- no-connect marks 2 -> 4
Other:
- note added: "Mounting holes for screws"
- moved on the sheet: P2, P3, P5, P6, R5, R6
