File: kicad-v7.0.9/signalization-by-fireplace/v1.0_v1.0/signalization-by-fireplace.kicad_sch (KiCad schematic)
At the start: 104 parts, among them J1 2x1x4_idc_lsa, J2 DG301-5.0-3P12, J3 54601-908WPLF, J4 2x1x4_idc_lsa, J5 DG390-5.0-02P-12-00A(H), J6 DG301-5.0-02P-12-00A(H), P1 1x4_pin_socket, P10 1x2_pin_header, P11 1x2_pin_header, P12 1x3_pin_header, P13 1x3_pin_header, P14 1x3_pin_header, P15 1x3_pin_header, P2 1x2_pin_header, P3 1x2_pin_header, P4 1x2_pin_header, P5 1x2_pin_header, P6 1x2_pin_header, P7 1x2_pin_header, P8 1x2_pin_header, P9 1x2_pin_header, Q1 BSS138P, Q2 BSS138P, Q3 BSS138P, Q4 BSS138P, Q6 YJL3415A, U1 PCA9615, U2 AP2210N-3.3TRG1, U3 MAX31850K, U4 TPS26600

Commit message: Signalization by fireplace. Change library. Small changes in schematic a PCB.
Parts:
- added H1, H11, H2, H3, H4, H5, H6: mounting_hole_pad_3.2x6mm, mounting_hole_pad_rl:mounting_hole_pad_3.2x6mm, symbol mounting_hole_pad_rl:mounting_hole_pad_3.2x6mm
- added H10, H7, H8, H9: mounting_hole_pad_3.2x5mm, mounting_hole_pad_rl:mounting_hole_pad_3.2x5mm, symbol mounting_hole_pad_rl:mounting_hole_pad_3.2x5mm
- C1, C10, C11, C12, C13, C14, C15, C2, C3, C4, C5, C6, C7, C8, C9: symbol passive_component_rl:capacitor -> capacitor_smd_rl:c_1206
- D1, D10, D14, D15, D2, D3, D8, D9: symbol diode_rl:undir_transil -> transil_diode_smd_rl:UCLAMP0501H.TCT
- D11: symbol diode_rl:bidir_transil -> transil_diode_smd_rl:ESD3B5V0WS
- D12: symbol diode_rl:DS9503_us -> transil_diode_smd_rl:DS9503_us
- D13: value OSB5SAA6A1A -> OSR5PAA6A1A; symbol diode_rl:LED -> led_tht_rl:OSR5PAA6A1A
- D16: symbol diode_rl:LED -> led_tht_rl:OSO5PAA6A1A
- D17: symbol diode_rl:ESD16VHYFHT116 -> transil_diode_smd_rl:ESD16VHYFHT116
- D18: value OSR5PAA6A1A -> OSB5SAA6A1A; symbol diode_rl:LED -> led_tht_rl:OSB5SAA6A1A
- D20: symbol diode_rl:LED -> led_tht_rl:LL-503VC1E-4C
- D22: symbol diode_rl:bidir_transil -> transil_diode_smd_rl:SMCJ5.0CA-13-F
- D4, D5, D6: symbol diode_rl:DS9503_us -> diode_smd_rl:DS9503_us
- D7: symbol diode_rl:SMDA05CDR2G -> transil_diode_smd_rl:SMDA05CDR2G
- J2: value DG301-5.0-3P12 -> EBBA-03-C-SS-BU; footprint terminal_block_tht_rl:DG301-5.0-03P-12-00A(H) -> terminal_block_tht_rl:EBBA-03-C-SS-BU; symbol connector_rl:1x3_screw_term_block -> terminal_block_tht_rl:EBBA-03-C-SS-BU
- J3: symbol connector_rl:rj45 -> connector_rj45_tht_rl:54601-908WPLF
- J5: value DG390-5.0-02P-12-00A(H) -> DG390-5.0; symbol connector_rl:1x2_screw_term_block -> terminal_block_tht_rl:DG390-5.0
- J6: value DG301-5.0-02P-12-00A(H) -> EBBA-02-C-SS-BU; footprint terminal_block_tht_rl:DG301-5.0-02P-12-00A(H) -> terminal_block_tht_rl:EBBA-02-C-SS-BU; symbol connector_rl:1x2_screw_term_block -> terminal_block_tht_rl:EBBA-02-C-SS-BU
- L1, L2: value 470R/1A -> BLM31KN471BH1L; symbol passive_component_rl:inductor -> ferrite_bead_smd_rl:BLM31KN471BH1L
- P1: value 1x4_pin_socket -> DS1023-1-4S21; symbol connector_rl:1x4_pin_socket -> connector_tht_pin_socket_2.54mm_rl:DS1023-1-4S21
- P10, P11, P2, P3, P4, P5, P6, P7, P8, P9: value 1x2_pin_header -> DS1021-1-2SF11-B; symbol connector_rl:1x2_pin_header -> connector_tht_pin_header_2.54mm_rl:DS1021-1-2SF11-B
- P12, P13, P14, P15: value 1x3_pin_header -> DS1021-1-3SF11-B; symbol connector_rl:1x3_pin_header -> connector_tht_pin_header_2.54mm_rl:DS1021-1-3SF11-B
- Q1, Q2, Q3, Q4: symbol signalization-by-fireplace-rescue:n_mosfet_gsd-unipolar_transistor_rl -> unipolar_transistor_smd_rl:BSS138P
- Q6: symbol signalization-by-fireplace-rescue:p_mosfet_gsd-unipolar_transistor_rl -> unipolar_transistor_smd_rl:YJL3415A
- R1, R10, R11, R12, R13, R14, R15, R16, R17, R18, R19, R2, R20, R21, R22, R23, R24, R25, R26, R27, R28, R3, R30, R31, R32, R33, R34, R35, R37, R38, R4, R5, R6, R7, R8, R9: symbol passive_component_rl:resistor_us -> resistor_smd_rl:r_1206_us
- R29: footprint trimmer_tht_rl:trimmer_t93yb -> trimmer_tht_rl:T93YB; symbol passive_component_rl:resistor_variable_us -> trimmer_tht_rl:T93YB; Manufacturer (none) -> Vishay
- U1: Manufacturer (none) -> NXP Semiconductors
- U2: symbol power_management_rl:XC6206P332MR-G -> low_dropout_regulator_rl:AP2210N-3.3TRG1
- U3: symbol thermocouple_rl:MAX31850K_rl -> thermocouple_rl:MAX31850K; Manufacturer (none) -> Maxim integrated
- U4: Manufacturer (none) -> Texas Instruments
Connections:
- no-connect marks 6 -> 17
Other:
- note added: "Mounting holes"
- note added: "Mounting holes for screws"
- note removed: "BLM31KN471BH1L"
- moved on the sheet: P10, P11, P8, P9, Q1, Q2, Q3, Q4, Q6, R16, R17, R18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
