File: kicad-v7.0.9/central-control-unit/central-control-unit/1-wire-bus.kicad_sch (KiCad schematic)
At the start: 116 parts, among them P25 10129380-902001BLF, P27 10129380-902001BLF, P29 10129380-902001BLF, P31 10129380-902001BLF, P33 10129380-902001BLF, P35 10129380-902001BLF, P36 10129380-902001BLF, P37 10129380-902001BLF, P38 10129380-902001BLF, P39 10129380-902001BLF, P40 10129380-902001BLF, P44 10129380-902001BLF, P45 95278-101A20LF, P46 95278-101A20LF, P47 10129380-902001BLF, P49 10129380-902001BLF, P51 10129380-902001BLF, P53 10129380-902001BLF, P55 10129380-902001BLF, P57 10129380-902001BLF, P58 10129380-902001BLF, P59 10129380-902001BLF, P60 10129380-902001BLF, Q39 PMV213SN,215, Q40 PMV213SN,215, Q41 PMV213SN,215, Q42 PMV213SN,215, Q43 PMV213SN,215, Q44 PMV213SN,215, Q45 PMV213SN,215, Q46 PMV213SN,215, Q47 PMV213SN,215, Q48 PMV213SN,215, Q49 PMV213SN,215, Q58 BXT600P03M, Q59 BXT600P03M, Q60 BXT600P03M, Q61 BXT600P03M, Q62 BXT600P03M, Q63 BXT600P03M, Q64 BXT600P03M, Q65 BXT600P03M, Q66 BXT600P03M, Q67 BXT600P03M, Q68 BXT600P03M, U23 TXS0108EPWR, U24 TXS0108EPWR

Commit message: Change components form library. Adding of BOM. Change folder structure.
Parts:
- P25, P27, P29, P31, P33, P35, P36, P37, P38, P39, P40, P44, P47, P49, P51, P53, P55, P57, P58, P59, P60: footprint connector_smd_pinheader_2.54mm_rl:1x2_pinheader_2.54mm_vertical -> connector_pin_header_2.54mm_smd_rl:1x2_pin_header_2.54mm_vertical; symbol connector_smd_pin_header_2.54mm_rl:10129380-902001BLF -> connector_pin_header_2.54mm_smd_rl:10129380-902001BLF
- P45, P46: footprint connector_smd_pinheader_2.54mm_rl:2x10_pinheader_2.54mm_vertical -> connector_pin_header_2.54mm_smd_rl:2x10_pin_header_2.54mm_vertical; symbol connector_smd_pin_header_2.54mm_rl:95278-101A20LF -> connector_pin_header_2.54mm_smd_rl:95278-101A20LF
