File: kicad-v7.0.9/central-control-unit/central-control-unit/central-control-unit.kicad_sch (KiCad schematic)
At the start: 24 parts, among them J4 EBBA-02-C-SS-BU, P1 95293-101A03LF, P2 95293-101A03LF, P26 DS1023-1-4S21, P28 molex_kk_254_1x02_2.54mm_2211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, P3 95293-101A03LF, P30 molex_kk_254_1x02_2.54mm_2211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, Q56 YJD20N06A, Q57 YJD20N06A, U8 MCP23S17-E/SP

Commit message: Change components form library. Adding of BOM. Change folder structure.
Parts:
- P1, P2, P3: footprint connector_smd_pinheader_2.54mm_rl:1x3_pinheader_2.54mm_vertical -> connector_pin_header_2.54mm_smd_rl:1x3_pin_header_2.54mm_vertical; symbol connector_smd_pin_header_2.54mm_rl:95293-101A03LF -> connector_pin_header_2.54mm_smd_rl:95293-101A03LF
- P26: footprint connector_tht_pinsocket_2.54mm_rl:1x4_pinsocket_2.54mm_vertical_8.5mm -> connector_pin_socket_2.54mm_tht_rl:1x4_pin_socket_2.54mm_vertical_8.5mm; symbol connector_tht_pin_socket_2.54mm_rl:DS1023-1-4S21 -> connector_pin_socket_2.54mm_tht_rl:DS1023-1-4S21
Changed lines of the file:
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@@
     )
   )
-  (symbol (lib_id "connector_tht_pin_socket_2.54mm_rl:DS1023-1-4S21") (at 90.17 44.45 0) (unit 1)
+  (symbol (lib_id "connector_pin_socket_2.54mm_tht_rl:DS1023-1-4S21") (at 90.17 44.45 0) (unit 1)
     (in_bom yes) (on_board yes) (dnp no)
     (property "Reference" "P26" (at 85.09 41.91 0)
@@
       (effects (font (size 1.27 1.27)))
     )
-    (property "Footprint" "connector_tht_pinsocket_2.54mm_rl:1x4_pinsocket_2.54mm_vertical_8.5mm" (at 90.17 36.83 0)
+    (property "Footprint" "connector_pin_socket_2.54mm_tht_rl:1x4_pin_socket_2.54mm_vertical_8.5mm" (at 90.17 36.83 0)
       (effects (font (size 1.27 1.27)) hide)
     )
@@
     )
   )
-  (symbol (lib_id "connector_smd_pin_header_2.54mm_rl:95293-101A03LF") (at 284.48 189.23 90) (unit 1)
+  (symbol (lib_id "connector_pin_header_2.54mm_smd_rl:95293-101A03LF") (at 284.48 189.23 90) (unit 1)
     (in_bom yes) (on_board yes) (dnp no)
     (property "Reference" "P1" (at 286.1818 180.975 90)
@@
       (effects (font (size 1.27 1.27)))
     )
-    (property "Footprint" "connector_smd_pinheader_2.54mm_rl:1x3_pinheader_2.54mm_vertical" (at 276.86 189.23 0)
+    (property "Footprint" "connector_pin_header_2.54mm_smd_rl:1x3_pin_header_2.54mm_vertical" (at 276.86 189.23 0)
       (effects (font (size 1.27 1.27)) hide)
     )
@@
     )
   )
-  (symbol (lib_id "connector_smd_pin_header_2.54mm_rl:95293-101A03LF") (at 307.34 189.23 90) (unit 1)
+  (symbol (lib_id "connector_pin_header_2.54mm_smd_rl:95293-101A03LF") (at 307.34 189.23 90) (unit 1)
     (in_bom yes) (on_board yes) (dnp no)
     (property "Reference" "P2" (at 309.0418 180.975 90)
@@
       (effects (font (size 1.27 1.27)))
     )
-    (property "Footprint" "connector_smd_pinheader_2.54mm_rl:1x3_pinheader_2.54mm_vertical" (at 299.72 189.23 0)
+    (property "Footprint" "connector_pin_header_2.54mm_smd_rl:1x3_pin_header_2.54mm_vertical" (at 299.72 189.23 0)
       (effects (font (size 1.27 1.27)) hide)
     )
@@
     )
   )
-  (symbol (lib_id "connector_smd_pin_header_2.54mm_rl:95293-101A03LF") (at 330.2 189.23 90) (unit 1)
+  (symbol (lib_id "connector_pin_header_2.54mm_smd_rl:95293-101A03LF") (at 330.2 189.23 90) (unit 1)
     (in_bom yes) (on_board yes) (dnp no)
     (property "Reference" "P3" (at 331.9018 180.975 90)
@@
       (effects (font (size 1.27 1.27)))
     )
-    (property "Footprint" "connector_smd_pinheader_2.54mm_rl:1x3_pinheader_2.54mm_vertical" (at 322.58 189.23 0)
-      (effects (font (size 1.27 1.27)) hide)
-    )
+    (property "Footprint" "connector_pin_header_2.54mm_smd_rl:1x3_pin_header_2.54mm_vertical" (at 322.58 189.23 0)
+      (effects (font (size 1.27 1.27)) hide)
+    )
