File: kicad-v7.0.9/central-control-unit/central-control-unit/connectors.kicad_sch (KiCad schematic)
At the start: 112 parts, among them J17 1x4_idc_lsa, J18 1x4_idc_lsa, J19 1x4_idc_lsa, J20 1x4_idc_lsa, J24 1x4_idc_lsa, J27 1x4_idc_lsa, J28 1x4_idc_lsa, J29 1x4_idc_lsa, J30 1x4_idc_lsa, J31 1x4_idc_lsa, J32 1x4_idc_lsa, J33 1x4_idc_lsa, J34 1x4_idc_lsa, J38 1x4_idc_lsa, J39 1x4_idc_lsa, J40 1x4_idc_lsa, J41 1x4_idc_lsa, J42 1x4_idc_lsa, J45 1x4_idc_lsa, J46 1x4_idc_lsa, J47 EBBA-03-C-SS-BU, J48 EBBA-03-C-SS-BU, J49 EBBA-03-C-SS-BU, J50 EBBA-03-C-SS-BU, J51 EBBA-03-C-SS-BU, J52 EBBA-03-C-SS-BU, P101 95293-101A03LF, P102 95293-101A03LF, P103 95293-101A03LF, P104 95293-101A03LF, P105 95293-101A03LF, P106 95293-101A03LF, P107 95293-101A03LF, P108 95293-101A03LF, P109 95293-101A03LF, P110 95293-101A03LF, P111 95293-101A03LF, P112 95293-101A03LF, Q50 PMV213SN,215, Q51 PMV213SN,215, Q52 PMV213SN,215, Q53 PMV213SN,215, Q54 PMV213SN,215, Q55 PMV213SN,215, U26 TXS0108EPWR, U27 TLP2345, U28 TLP2345, U29 TLP2345, U30 TLP2345, U31 TLP2345, U32 TLP2345

Commit message: Change components form library. Adding of BOM. Change folder structure.
Parts:
- J17, J18, J19, J20, J24, J27, J28, J29, J30, J31, J32, J33, J34, J38, J39, J40, J41, J42, J45, J46: footprint connector_rl:1x4_idc_lsa_connector_general -> connector_idc_lsa_tht_rl:1x4_idc_lsa_connector_general; symbol connector_rl:1x4_idc_lsa -> connector_idc_lsa_tht_rl:1x4_idc_lsa
- P101, P102, P103, P104, P105, P106, P107, P108, P109, P110, P111, P112: footprint connector_smd_pinheader_2.54mm_rl:1x3_pinheader_2.54mm_vertical -> connector_pin_header_2.54mm_smd_rl:1x3_pin_header_2.54mm_vertical; symbol connector_smd_pin_header_2.54mm_rl:95293-101A03LF -> connector_pin_header_2.54mm_smd_rl:95293-101A03LF
