File: kicad-v7.0.9/central-control-unit/central-control-unit/pin-headers.kicad_sch (KiCad schematic)
At the start: 5 parts, among them P115 DS1023-2-20S21, P116 DS1021-2-20SF11-B, P4 DS1023-1-20S21

Commit message: Change components form library. Adding of BOM. Change folder structure.
Parts:
- P115: symbol connector_tht_pin_socket_2.54mm_rl:DS1023-2-20S21 -> connector_pin_socket_2.54mm_tht_rl:DS1023-2-20S21
- P116: footprint connector_tht_pinheader_2.54mm_rl:2x20_pinheader_2.54mm_vertical -> connector_pin_header_2.54mm_tht_rl:2x20_pin_header_2.54mm_vertical; symbol connector_tht_pin_header_2.54mm_rl:DS1021-2-20SF11-B -> connector_pin_header_2.54mm_tht_rl:DS1021-2-20SF11-B
- P4: footprint connector_tht_pinsocket_2.54mm_rl:1x20_pinsocket_2.54mm_vertical_8.5mm -> connector_pin_socket_2.54mm_tht_rl:1x20_pin_socket_2.54mm_vertical_8.5mm; symbol connector_tht_pin_socket_2.54mm_rl:DS1023-1-20S21 -> connector_pin_socket_2.54mm_tht_rl:DS1023-1-20S21
Changed lines of the file:
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@@
     )
   )
-  (symbol (lib_id "connector_tht_pin_socket_2.54mm_rl:DS1023-1-20S21") (at 31.75 147.32 90) (mirror x) (unit 1)
+  (symbol (lib_id "connector_pin_socket_2.54mm_tht_rl:DS1023-1-20S21") (at 31.75 147.32 90) (mirror x) (unit 1)
     (in_bom yes) (on_board yes) (dnp no)
     (property "Reference" "P4" (at 31.75 120.65 90)
@@
       (effects (font (size 1.27 1.27)))
     )
-    (property "Footprint" "connector_tht_pinsocket_2.54mm_rl:1x20_pinsocket_2.54mm_vertical_8.5mm" (at 24.13 147.32 0)
+    (property "Footprint" "connector_pin_socket_2.54mm_tht_rl:1x20_pin_socket_2.54mm_vertical_8.5mm" (at 24.13 147.32 0)
       (effects (font (size 1.27 1.27)) hide)
     )
@@
     )
   )
-  (symbol (lib_id "connector_tht_pin_socket_2.54mm_rl:DS1023-2-20S21") (at 113.03 53.34 270) (unit 1)
+  (symbol (lib_id "connector_pin_socket_2.54mm_tht_rl:DS1023-2-20S21") (at 113.03 53.34 270) (unit 1)
     (in_bom yes) (on_board yes) (dnp no)
     (property "Reference" "P115" (at 113.03 26.67 90)
@@
     )
   )
-  (symbol (lib_id "connector_tht_pin_header_2.54mm_rl:DS1021-2-20SF11-B") (at 222.25 114.3 270) (unit 1)
+  (symbol (lib_id "connector_pin_header_2.54mm_tht_rl:DS1021-2-20SF11-B") (at 222.25 114.3 270) (unit 1)
     (in_bom yes) (on_board yes) (dnp no)
     (property "Reference" "P116" (at 222.25 87.63 90)
@@
       (effects (font (size 1.27 1.27)))
     )
-    (property "Footprint" "connector_tht_pinheader_2.54mm_rl:2x20_pinheader_2.54mm_vertical" (at 237.49 114.3 0)
-      (effects (font (size 1.27 1.27)) hide)
-    )
+    (property "Footprint" "connector_pin_header_2.54mm_tht_rl:2x20_pin_header_2.54mm_vertical" (at 237.49 114.3 0)
+      (effects (font (size 1.27 1.27)) hide)
+    )
