File: kicad-v7.0.9/central-control-unit/central-control-unit/relays-outputs.kicad_sch (KiCad schematic)
At the start: 188 parts, among them J10 EBBA-02-C-SS-BU, J11 EBBA-02-C-SS-BU, J12 AKZ770_3-5.08-V-GREEN, J13 EBBA-02-C-SS-BU, J14 EBBA-02-C-SS-BU, J15 EBBA-02-C-SS-BU, J16 EBBA-02-C-SS-BU, J6 EBBA-02-C-SS-BU, J7 EBBA-02-C-SS-BU, J8 EBBA-02-C-SS-BU, J9 EBBA-02-C-SS-BU, P10 95293-101A03LF, P11 95293-101A03LF, P12 95293-101A03LF, P13 95293-101A03LF, P14 95293-101A03LF, P15 95293-101A03LF, P16 95293-101A03LF, P17 95293-101A03LF, P18 95293-101A03LF, P19 95293-101A03LF, P20 95293-101A03LF, P21 95293-101A03LF, P22 95293-101A03LF, P23 95293-101A03LF, P24 95293-101A03LF, P5 95293-101A03LF, P6 95293-101A03LF, P7 95293-101A03LF, P8 95293-101A03LF, P9 95293-101A03LF, Q23 AOD458, Q24 AOD458, Q25 AOD458, Q26 AOD458, Q27 AOD458, Q28 AOD458, Q29 PMV213SN,215, Q30 PMV213SN,215, Q31 PMV213SN,215, Q32 PMV213SN,215, Q33 PMV213SN,215, Q34 PMV213SN,215, Q35 AOD458, Q36 AOD458, Q37 AOD458, Q38 AOD458, Q69 PMV213SN,215, Q70 PMV213SN,215, Q71 PMV213SN,215, Q72 PMV213SN,215, Q73 PMV213SN,215, Q74 PMV213SN,215, U13 TLP2345, U14 TLP2345, U15 TLP2345, U16 TLP2345, U17 TLP2345, U18 TLP2345, U19 TLP2345, U20 TLP2345, U21 TLP2345, U22 TLP2345

Commit message: Change components form library. Adding of BOM. Change folder structure.
Parts:
- P10, P11, P12, P13, P14, P15, P16, P17, P18, P19, P20, P21, P22, P23, P24, P5, P6, P7, P8, P9: footprint connector_smd_pinheader_2.54mm_rl:1x3_pinheader_2.54mm_vertical -> connector_pin_header_2.54mm_smd_rl:1x3_pin_header_2.54mm_vertical; symbol connector_smd_pin_header_2.54mm_rl:95293-101A03LF -> connector_pin_header_2.54mm_smd_rl:95293-101A03LF
