File: kicad-v7.0.9/central-control-unit/power-in-usb-c/power-in-usb-c.kicad_sch (KiCad schematic)
At the start: 5 parts, among them P1 DS1021-1-4SF11-B

Commit message: Change components form library. Adding of BOM.
Parts:
- P1: footprint connector_tht_pinheader_2.54mm_rl:1x4_pinheader_2.54mm_vertical -> connector_pin_header_2.54mm_tht_rl:1x4_pin_header_2.54mm_vertical; symbol connector_tht_pin_header_2.54mm_rl:DS1021-1-4SF11-B -> connector_pin_header_2.54mm_tht_rl:DS1021-1-4SF11-B
Changed lines of the file:
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@@
     (stroke (width 0) (type default))
   )
-  (symbol (lib_id "connector_tht_pin_header_2.54mm_rl:DS1021-1-4SF11-B") (at 124.46 50.8 0) (unit 1)
+  (symbol (lib_id "connector_pin_header_2.54mm_tht_rl:DS1021-1-4SF11-B") (at 124.46 50.8 0) (unit 1)
     (in_bom yes) (on_board yes) (dnp no)
     (property "Reference" "P1" (at 130.5052 51.3334 0)
@@
       (effects (font (size 1.27 1.27)))
     )
-    (property "Footprint" "connector_tht_pinheader_2.54mm_rl:1x4_pinheader_2.54mm_vertical" (at 124.46 43.18 0)
+    (property "Footprint" "connector_pin_header_2.54mm_tht_rl:1x4_pin_header_2.54mm_vertical" (at 124.46 43.18 0)
       (effects (font (size 1.27 1.27)) hide)
     )
