File: kicad-v7.0.9/central-control-unit/switches-with-lcd-display/switches-with-lcd-display.kicad_sch (KiCad schematic)
At the start: 80 parts, among them P1 112-A-S-S-20-G-38mm, P2 95293-101A03LF, P3 95293-101A03LF, P4 95293-101A03LF, P6 95293-101A03LF, Q1 PMV213SN,215, SW1 SMTS-102-2C2T, SW10 SMTS-102-2C2T, SW2 SMTS-102-2C2T, SW3 SMTS-102-2C2T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

Commit message: Change components form library. Adding of BOM.
Parts:
- P1: footprint connector_tht_pinheader_2.54mm_rl:1x20_pinheader_2.54mm_vertical -> connector_pin_header_2.54mm_tht_rl:1x20_pin_header_2.54mm_vertical; symbol connector_tht_pin_header_2.54mm_rl:112-A-S-S-20-G-38mm -> connector_pin_header_2.54mm_tht_rl:112-A-S-S-20-G-38mm
- P2, P3, P4, P6: footprint connector_smd_pinheader_2.54mm_rl:1x3_pinheader_2.54mm_vertical -> connector_pin_header_2.54mm_smd_rl:1x3_pin_header_2.54mm_vertical; symbol connector_smd_pin_header_2.54mm_rl:95293-101A03LF -> connector_pin_header_2.54mm_smd_rl:95293-101A03LF
Changed lines of the file:
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@@
       (effects (font (size 1.27 1.27)) (justify right))
     )
-    (property "Footprint" "switch_tht_rl:SMTS-102-2C2T" (at 44.45 247.65 0)
+    (property "Footprint" "switch_tht_rl:SMTS-102-2C2T" (at 31.75 248.92 0)
       (effects (font (size 1.27 1.27)) hide)
     )
-    (property "Datasheet" "https://www.gme.cz/data/attachments/dsh.631-528.1.pdf" (at 44.45 247.65 0)
+    (property "Datasheet" "https://www.gme.cz/data/attachments/dsh.631-528.1.pdf" (at 34.29 248.92 0)
       (effects (font (size 1.27 1.27)) hide)
     )
@@
     )
   )
-  (symbol (lib_id "connector_tht_pin_header_2.54mm_rl:112-A-S-S-20-G-38mm") (at 209.55 53.34 90) (mirror x) (unit 1)
+  (symbol (lib_id "connector_pin_header_2.54mm_tht_rl:112-A-S-S-20-G-38mm") (at 209.55 53.34 90) (mirror x) (unit 1)
     (in_bom yes) (on_board yes) (dnp no)
     (property "Reference" "P1" (at 209.55 26.67 90)
@@
       (effects (font (size 1.27 1.27)))
     )
-    (property "Footprint" "connector_tht_pinheader_2.54mm_rl:1x20_pinheader_2.54mm_vertical" (at 209.296 48.26 0)
+    (property "Footprint" "connector_pin_header_2.54mm_tht_rl:1x20_pin_header_2.54mm_vertical" (at 201.93 53.34 0)
       (effects (font (size 1.27 1.27)) hide)
     )
@@
       (effects (font (size 1.27 1.27)) (justify right))
     )
-    (property "Footprint" "switch_tht_rl:SMTS-102-2C2T" (at 182.88 198.12 0)
+    (property "Footprint" "switch_tht_rl:SMTS-102-2C2T" (at 170.18 199.39 0)
       (effects (font (size 1.27 1.27)) hide)
     )
-    (property "Datasheet" "https://www.gme.cz/data/attachments/dsh.631-528.1.pdf" (at 182.88 198.12 0)
+    (property "Datasheet" "https://www.gme.cz/data/attachments/dsh.631-528.1.pdf" (at 172.72 199.39 0)
       (effects (font (size 1.27 1.27)) hide)
     )
@@
       (effects (font (size 1.27 1.27)) (justify right))
     )
-    (property "Footprint" "switch_tht_rl:SMTS-102-2C2T" (at 182.88 247.65 0)
+    (property "Footprint" "switch_tht_rl:SMTS-102-2C2T" (at 170.18 248.92 0)
       (effects (font (size 1.27 1.27)) hide)
     )
-    (property "Datasheet" "https://www.gme.cz/data/attachments/dsh.631-528.1.pdf" (at 182.88 247.65 0)
+    (property "Datasheet" "https://www.gme.cz/data/attachments/dsh.631-528.1.pdf" (at 172.72 248.92 0)
       (effects (font (size 1.27 1.27)) hide)
     )
@@
       (effects (font (size 1.27 1.27)) (justify right))
     )
-    (property "Footprint" "switch_tht_rl:SMTS-102-2C2T" (at 327.66 217.17 0)
+    (property "Footprint" "switch_tht_rl:SMTS-102-2C2T" (at 314.96 218.44 0)
       (effects (font (size 1.27 1.27)) hide)
     )
-    (property "Datasheet" "https://www.gme.cz/data/attachments/dsh.631-528.1.pdf" (at 327.66 217.17 0)
+    (property "Datasheet" "https://www.gme.cz/data/attachments/dsh.631-528.1.pdf" (at 317.5 218.44 0)
       (effects (font (size 1.27 1.27)) hide)
     )
@@
       (effects (font (size 1.27 1.27)) (justify right))
     )
-    (property "Footprint" "switch_tht_rl:SMTS-102-2C2T" (at 222.25 151.13 0)
+    (property "Footprint" "switch_tht_rl:SMTS-102-2C2T" (at 209.55 152.4 0)
       (effects (font (size 1.27 1.27)) hide)
     )
-    (property "Datasheet" "https://www.gme.cz/data/attachments/dsh.631-528.1.pdf" (at 222.25 151.13 0)
+    (property "Datasheet" "https://www.gme.cz/data/attachments/dsh.631-528.1.pdf" (at 212.09 152.4 0)
       (effects (font (size 1.27 1.27)) hide)
     )
@@
       (effects (font (size 1.27 1.27)) (justify right))
     )
-    (property "Footprint" "switch_tht_rl:SMTS-102-2C2T" (at 328.93 29.21 0)
+    (property "Footprint" "switch_tht_rl:SMTS-102-2C2T" (at 316.23 30.48 0)
       (effects (font (size 1.27 1.27)) hide)
     )
-    (property "Datasheet" "https://www.gme.cz/data/attachments/dsh.631-528.1.pdf" (at 328.93 29.21 0)
+    (property "Datasheet" "https://www.gme.cz/data/attachments/dsh.631-528.1.pdf" (at 318.77 30.48 0)
       (effects (font (size 1.27 1.27)) hide)
     )
@@
       (effects (font (size 1.27 1.27)) (justify right))
     )
-    (property "Footprint" "switch_tht_rl:SMTS-102-2C2T" (at 327.66 77.47 0)
+    (property "Footprint" "switch_tht_rl:SMTS-102-2C2T" (at 314.96 78.74 0)
       (effects (font (size 1.27 1.27)) hide)
     )
-    (property "Datasheet" "https://www.gme.cz/data/attachments/dsh.631-528.1.pdf" (at 327.66 77.47 0)
+    (property "Datasheet" "https://www.gme.cz/data/attachments/dsh.631-528.1.pdf" (at 317.5 78.74 0)
       (effects (font (size 1.27 1.27)) hide)
     )
@@
       (effects (font (size 1.27 1.27)) (justify right))
     )
-    (property "Footprint" "switch_tht_rl:SMTS-102-2C2T" (at 327.66 124.46 0)
+    (property "Footprint" "switch_tht_rl:SMTS-102-2C2T" (at 314.96 125.73 0)
       (effects (font (size 1.27 1.27)) hide)
     )
-    (property "Datasheet" "https://www.gme.cz/data/attachments/dsh.631-528.1.pdf" (at 327.66 124.46 0)
+    (property "Datasheet" "https://www.gme.cz/data/attachments/dsh.631-528.1.pdf" (at 317.5 125.73 0)
       (effects (font (size 1.27 1.27)) hide)
     )
@@
       (effects (font (size 1.27 1.27)) (justify right))
     )
-    (property "Footprint" "switch_tht_rl:SMTS-102-2C2T" (at 327.66 170.18 0)
+    (property "Footprint" "switch_tht_rl:SMTS-102-2C2T" (at 314.96 171.45 0)
       (effects (font (size 1.27 1.27)) hide)
     )
-    (property "Datasheet" "https://www.gme.cz/data/attachments/dsh.631-528.1.pdf" (at 327.66 170.18 0)
+    (property "Datasheet" "https://www.gme.cz/data/attachments/dsh.631-528.1.pdf" (at 317.5 171.45 0)
       (effects (font (size 1.27 1.27)) hide)
     )
@@
     )
   )
-  (symbol (lib_id "connector_smd_pin_header_2.54mm_rl:95293-101A03LF") (at 33.02 113.03 90) (unit 1)
+  (symbol (lib_id "connector_pin_header_2.54mm_smd_rl:95293-101A03LF") (at 33.02 113.03 90) (unit 1)
     (in_bom yes) (on_board yes) (dnp no)
     (property "Reference" "P2" (at 34.7218 104.775 90)
@@
       (effects (font (size 1.27 1.27)))
     )
-    (property "Footprint" "connector_smd_pinheader_2.54mm_rl:1x3_pinheader_2.54mm_vertical" (at 25.4 113.03 0)
+    (property "Footprint" "connector_pin_header_2.54mm_smd_rl:1x3_pin_header_2.54mm_vertical" (at 25.4 113.03 0)
       (effects (font (size 1.27 1.27)) hide)
     )
@@
     )
   )
-  (symbol (lib_id "connector_smd_pin_header_2.54mm_rl:95293-101A03LF") (at 55.88 113.03 90) (unit 1)
+  (symbol (lib_id "connector_pin_header_2.54mm_smd_rl:95293-101A03LF") (at 55.88 113.03 90) (unit 1)
     (in_bom yes) (on_board yes) (dnp no)
     (property "Reference" "P3" (at 57.5818 104.775 90)
@@
       (effects (font (size 1.27 1.27)))
     )
-    (property "Footprint" "connector_smd_pinheader_2.54mm_rl:1x3_pinheader_2.54mm_vertical" (at 48.26 113.03 0)
+    (property "Footprint" "connector_pin_header_2.54mm_smd_rl:1x3_pin_header_2.54mm_vertical" (at 48.26 113.03 0)
       (effects (font (size 1.27 1.27)) hide)
     )
@@
     )
   )
-  (symbol (lib_id "connector_smd_pin_header_2.54mm_rl:95293-101A03LF") (at 78.74 113.03 90) (unit 1)
+  (symbol (lib_id "connector_pin_header_2.54mm_smd_rl:95293-101A03LF") (at 78.74 113.03 90) (unit 1)
     (in_bom yes) (on_board yes) (dnp no)
     (property "Reference" "P4" (at 80.4418 104.775 90)
@@
       (effects (font (size 1.27 1.27)))
     )
-    (property "Footprint" "connector_smd_pinheader_2.54mm_rl:1x3_pinheader_2.54mm_vertical" (at 71.12 113.03 0)
+    (property "Footprint" "connector_pin_header_2.54mm_smd_rl:1x3_pin_header_2.54mm_vertical" (at 71.12 113.03 0)
       (effects (font (size 1.27 1.27)) hide)
     )
@@
     )
   )
-  (symbol (lib_id "connector_smd_pin_header_2.54mm_rl:95293-101A03LF") (at 163.83 24.13 0) (unit 1)
+  (symbol (lib_id "connector_pin_header_2.54mm_smd_rl:95293-101A03LF") (at 163.83 24.13 0) (unit 1)
     (in_bom yes) (on_board yes) (dnp no)
     (property "Reference" "P6" (at 168.6052 24.6634 0)
@@
       (effects (font (size 1.27 1.27)))
     )
-    (property "Footprint" "connector_smd_pinheader_2.54mm_rl:1x3_pinheader_2.54mm_vertical" (at 163.83 16.51 0)
+    (property "Footprint" "connector_pin_header_2.54mm_smd_rl:1x3_pin_header_2.54mm_vertical" (at 163.83 16.51 0)
       (effects (font (size 1.27 1.27)) hide)
     )
@@
       (effects (font (size 1.27 1.27)) (justify right))
     )
-    (property "Footprint" "switch_tht_rl:SMTS-102-2C2T" (at 44.45 196.85 0)
+    (property "Footprint" "switch_tht_rl:SMTS-102-2C2T" (at 31.75 198.12 0)
       (effects (font (size 1.27 1.27)) hide)
     )
-    (property "Datasheet" "https://www.gme.cz/data/attachments/dsh.631-528.1.pdf" (at 44.45 196.85 0)
+    (property "Datasheet" "https://www.gme.cz/data/attachments/dsh.631-528.1.pdf" (at 34.29 198.12 0)
       (effects (font (size 1.27 1.27)) hide)
     )
