File: kicad-v7.0.9/signalization-by-fireplace/signalization-by-fireplace.kicad_sch (KiCad schematic)
At the start: 115 parts, among them J1 2x1x4_idc_lsa, J2 EBBA-03-C-SS-BU, J3 54601-908WPLF, J4 2x1x4_idc_lsa, J5 DG390-5.0, J6 EBBA-02-C-SS-BU, P1 DS1023-1-4S21, P10 DS1021-1-2SF11-B, P11 DS1021-1-2SF11-B, P12 DS1021-1-3SF11-B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

Commit message: Change of components from edited library. Change folder structure.
Parts:
- J3: footprint connector_rl:rj45_54601-908WPLF -> connector_rj45_tht_rl:54601-908WPLF
- P1: footprint connector_tht_pinsocket_2.54mm_rl:1x4_pinsocket_2.54mm_vertical_8.4mm -> connector_tht_pinsocket_2.54mm_rl:1x4_pinsocket_2.54mm_vertical_8.5mm
Changed lines of the file:
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@@
   (junction (at 96.52 72.39) (diameter 0) (color 0 0 0 0)
   )
-  (no_connect (at 318.77 64.77))
   (no_connect (at 318.77 38.1))
   (no_connect (at 344.17 133.35))
@@
   (no_connect (at 34.29 214.63))
   (no_connect (at 318.77 53.34))
+  (no_connect (at 318.77 68.58))
   (no_connect (at 321.31 130.81))
   (no_connect (at 318.77 60.96))
@@
       (effects (font (size 1.27 1.27)))
     )
-    (property "Footprint" "connector_rl:rj45_54601-908WPLF" (at 24.13 200.66 0)
+    (property "Footprint" "connector_rj45_tht_rl:54601-908WPLF" (at 24.13 200.66 0)
       (effects (font (size 1.27 1.27)) hide)
     )
@@
       (effects (font (size 1.27 1.27)))
     )
-    (property "Footprint" "connector_tht_pinsocket_2.54mm_rl:1x4_pinsocket_2.54mm_vertical_8.4mm" (at 36.83 124.46 0)
+    (property "Footprint" "connector_tht_pinsocket_2.54mm_rl:1x4_pinsocket_2.54mm_vertical_8.5mm" (at 36.83 124.46 0)
       (effects (font (size 1.27 1.27)) hide)
     )

Commit message: Change components form library. Adding of BOM.
Parts:
- J1, J4: footprint connector_rl:1x4_idc_lsa_connector_general -> connector_idc_lsa_tht_rl:1x4_idc_lsa_connector_general; symbol connector_rl:1x4_idc_lsa -> connector_idc_lsa_tht_rl:1x4_idc_lsa
- P1: footprint connector_tht_pinsocket_2.54mm_rl:1x4_pinsocket_2.54mm_vertical_8.5mm -> connector_pin_socket_2.54mm_tht_rl:1x4_pin_socket_2.54mm_vertical_8.5mm; symbol connector_tht_pin_socket_2.54mm_rl:DS1023-1-4S21 -> connector_pin_socket_2.54mm_tht_rl:DS1023-1-4S21
- P10, P11, P2, P3, P4, P5, P6, P7, P8, P9: footprint connector_tht_pinheader_2.54mm_rl:1x2_pinheader_2.54mm_vertical -> connector_pin_header_2.54mm_tht_rl:1x2_pin_header_2.54mm_vertical; symbol connector_tht_pin_header_2.54mm_rl:DS1021-1-2SF11-B -> connector_pin_header_2.54mm_tht_rl:DS1021-1-2SF11-B
- P12, P13, P14, P15: footprint connector_tht_pinheader_2.54mm_rl:1x3_pinheader_2.54mm_vertical -> connector_pin_header_2.54mm_tht_rl:1x3_pin_header_2.54mm_vertical; symbol connector_tht_pin_header_2.54mm_rl:DS1021-1-3SF11-B -> connector_pin_header_2.54mm_tht_rl:DS1021-1-3SF11-B
