File: kicad-v7.0.9/testing-board/testing-board.kicad_sch (KiCad schematic)
At the start: 39 parts, among them J1 54601-908WPLF, J2 EBBA-02-C-SS-BU, P1 DS1021-1-3SF11-B, P10 10129380-902001BLF, P11 10129380-902001BLF, P12 10129380-902001BLF, P13 10129380-902001BLF, P14 10129380-902001BLF, P2 DS1023-1-3S21, P3 DS1021-1-4SF11-B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

Commit message: Change of components from edited library. Change folder structure.
Parts:
- J1: footprint connector_rl:rj45_54601-908WPLF -> connector_rj45_tht_rl:54601-908WPLF
- P2: footprint connector_tht_pinsocket_2.54mm_rl:1x3_pinsocket_2.54mm_vertical_8.4mm -> connector_tht_pinsocket_2.54mm_rl:1x3_pinsocket_2.54mm_vertical_8.5mm
- P4: footprint connector_tht_pinsocket_2.54mm_rl:1x4_pinsocket_2.54mm_vertical_8.4mm -> connector_tht_pinsocket_2.54mm_rl:1x4_pinsocket_2.54mm_vertical_8.5mm
Changed lines of the file:
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@@
       (effects (font (size 1.27 1.27)))
     )
-    (property "Footprint" "connector_rl:rj45_54601-908WPLF" (at 33.02 45.72 0)
+    (property "Footprint" "connector_rj45_tht_rl:54601-908WPLF" (at 33.02 45.72 0)
       (effects (font (size 1.27 1.27)) hide)
     )
@@
       (effects (font (size 1.27 1.27)))
     )
-    (property "Footprint" "connector_tht_pinsocket_2.54mm_rl:1x3_pinsocket_2.54mm_vertical_8.4mm" (at 19.05 120.65 0)
+    (property "Footprint" "connector_tht_pinsocket_2.54mm_rl:1x3_pinsocket_2.54mm_vertical_8.5mm" (at 19.05 120.65 0)
       (effects (font (size 1.27 1.27)) hide)
     )
@@
       (effects (font (size 1.27 1.27)))
     )
-    (property "Footprint" "connector_tht_pinsocket_2.54mm_rl:1x4_pinsocket_2.54mm_vertical_8.4mm" (at 48.26 167.64 0)
-      (effects (font (size 1.27 1.27)) hide)
-    )
+    (property "Footprint" "connector_tht_pinsocket_2.54mm_rl:1x4_pinsocket_2.54mm_vertical_8.5mm" (at 48.26 167.64 0)
+      (effects (font (size 1.27 1.27)) hide)
+    )

Commit message: Change components form library. Adding of BOM.
Parts:
- P1: footprint connector_tht_pinheader_2.54mm_rl:1x3_pinheader_2.54mm_vertical -> connector_pin_header_2.54mm_tht_rl:1x3_pin_header_2.54mm_vertical; symbol connector_tht_pin_header_2.54mm_rl:DS1021-1-3SF11-B -> connector_pin_header_2.54mm_tht_rl:DS1021-1-3SF11-B
- P10, P11, P12, P13, P14, P5, P6, P7, P8, P9: footprint connector_smd_pinheader_2.54mm_rl:1x2_pinheader_2.54mm_vertical -> connector_pin_header_2.54mm_smd_rl:1x2_pin_header_2.54mm_vertical; symbol connector_smd_pin_header_2.54mm_rl:10129380-902001BLF -> connector_pin_header_2.54mm_smd_rl:10129380-902001BLF
- P2: footprint connector_tht_pinsocket_2.54mm_rl:1x3_pinsocket_2.54mm_vertical_8.5mm -> connector_pin_socket_2.54mm_tht_rl:1x3_pin_socket_2.54mm_vertical_8.5mm; symbol connector_tht_pin_socket_2.54mm_rl:DS1023-1-3S21 -> connector_pin_socket_2.54mm_tht_rl:DS1023-1-3S21
- P3: footprint connector_tht_pinheader_2.54mm_rl:1x4_pinheader_2.54mm_vertical -> connector_pin_header_2.54mm_tht_rl:1x4_pin_header_2.54mm_vertical; symbol connector_tht_pin_header_2.54mm_rl:DS1021-1-4SF11-B -> connector_pin_header_2.54mm_tht_rl:DS1021-1-4SF11-B
- P4: footprint connector_tht_pinsocket_2.54mm_rl:1x4_pinsocket_2.54mm_vertical_8.5mm -> connector_pin_socket_2.54mm_tht_rl:1x4_pin_socket_2.54mm_vertical_8.5mm; symbol connector_tht_pin_socket_2.54mm_rl:DS1023-1-4S21 -> connector_pin_socket_2.54mm_tht_rl:DS1023-1-4S21
Changed lines of the file:
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@@
     )
   )
-  (symbol (lib_id "connector_smd_pin_header_2.54mm_rl:10129380-902001BLF") (at 142.24 71.12 90) (unit 1)
+  (symbol (lib_id "connector_pin_header_2.54mm_smd_rl:10129380-902001BLF") (at 142.24 71.12 90) (unit 1)
     (in_bom yes) (on_board yes) (dnp no)
     (property "Reference" "P5" (at 138.43 69.85 90)
@@
       (effects (font (size 1.27 1.27)))
     )
-    (property "Footprint" "connector_smd_pinheader_2.54mm_rl:1x2_pinheader_2.54mm_vertical" (at 134.62 71.12 0)
+    (property "Footprint" "connector_pin_header_2.54mm_smd_rl:1x2_pin_header_2.54mm_vertical" (at 134.62 71.12 0)
       (effects (font (size 1.27 1.27)) hide)
     )
@@
     )
   )
-  (symbol (lib_id "connector_smd_pin_header_2.54mm_rl:10129380-902001BLF") (at 161.29 71.12 270) (mirror x) (unit 1)
+  (symbol (lib_id "connector_pin_header_2.54mm_smd_rl:10129380-902001BLF") (at 161.29 71.12 270) (mirror x) (unit 1)
     (in_bom yes) (on_board yes) (dnp no)
     (property "Reference" "P6" (at 165.1 69.85 90)
@@
       (effects (font (size 1.27 1.27)))
     )
-    (property "Footprint" "connector_smd_pinheader_2.54mm_rl:1x2_pinheader_2.54mm_vertical" (at 168.91 71.12 0)
+    (property "Footprint" "connector_pin_header_2.54mm_smd_rl:1x2_pin_header_2.54mm_vertical" (at 168.91 71.12 0)
       (effects (font (size 1.27 1.27)) hide)
     )
@@
     )
   )
-  (symbol (lib_id "connector_tht_pin_socket_2.54mm_rl:DS1023-1-3S21") (at 26.67 120.65 90) (unit 1)
+  (symbol (lib_id "connector_pin_socket_2.54mm_tht_rl:DS1023-1-3S21") (at 26.67 120.65 90) (unit 1)
     (in_bom yes) (on_board yes) (dnp no)
     (property "Reference" "P2" (at 26.67 115.57 90)
@@
       (effects (font (size 1.27 1.27)))
     )
-    (property "Footprint" "connector_tht_pinsocket_2.54mm_rl:1x3_pinsocket_2.54mm_vertical_8.5mm" (at 19.05 120.65 0)
+    (property "Footprint" "connector_pin_socket_2.54mm_tht_rl:1x3_pin_socket_2.54mm_vertical_8.5mm" (at 19.05 120.65 0)
       (effects (font (size 1.27 1.27)) hide)
     )
@@
     )
   )
-  (symbol (lib_id "connector_tht_pin_socket_2.54mm_rl:DS1023-1-4S21") (at 55.88 167.64 90) (unit 1)
+  (symbol (lib_id "connector_pin_socket_2.54mm_tht_rl:DS1023-1-4S21") (at 55.88 167.64 90) (unit 1)
     (in_bom yes) (on_board yes) (dnp no)
     (property "Reference" "P4" (at 55.88 161.29 90)
@@
       (effects (font (size 1.27 1.27)))
     )
-    (property "Footprint" "connector_tht_pinsocket_2.54mm_rl:1x4_pinsocket_2.54mm_vertical_8.5mm" (at 48.26 167.64 0)
+    (property "Footprint" "connector_pin_socket_2.54mm_tht_rl:1x4_pin_socket_2.54mm_vertical_8.5mm" (at 48.26 167.64 0)
       (effects (font (size 1.27 1.27)) hide)
     )
@@
     )
   )
-  (symbol (lib_id "connector_smd_pin_header_2.54mm_rl:10129380-902001BLF") (at 204.47 88.9 90) (unit 1)
+  (symbol (lib_id "connector_pin_header_2.54mm_smd_rl:10129380-902001BLF") (at 204.47 88.9 90) (unit 1)
     (in_bom yes) (on_board yes) (dnp no)
     (property "Reference" "P7" (at 200.66 87.63 90)
@@
       (effects (font (size 1.27 1.27)))
     )
-    (property "Footprint" "connector_smd_pinheader_2.54mm_rl:1x2_pinheader_2.54mm_vertical" (at 196.85 88.9 0)
+    (property "Footprint" "connector_pin_header_2.54mm_smd_rl:1x2_pin_header_2.54mm_vertical" (at 196.85 88.9 0)
       (effects (font (size 1.27 1.27)) hide)
     )
@@
     )
   )
-  (symbol (lib_id "connector_smd_pin_header_2.54mm_rl:10129380-902001BLF") (at 204.47 101.6 90) (unit 1)
+  (symbol (lib_id "connector_pin_header_2.54mm_smd_rl:10129380-902001BLF") (at 204.47 101.6 90) (unit 1)
     (in_bom yes) (on_board yes) (dnp no)
     (property "Reference" "P8" (at 200.66 99.06 90)
@@
       (effects (font (size 1.27 1.27)))
     )
-    (property "Footprint" "connector_smd_pinheader_2.54mm_rl:1x2_pinheader_2.54mm_vertical" (at 196.85 101.6 0)
+    (property "Footprint" "connector_pin_header_2.54mm_smd_rl:1x2_pin_header_2.54mm_vertical" (at 196.85 101.6 0)
       (effects (font (size 1.27 1.27)) hide)
     )
@@
     )
   )
-  (symbol (lib_id "connector_smd_pin_header_2.54mm_rl:10129380-902001BLF") (at 204.47 116.84 90) (unit 1)
+  (symbol (lib_id "connector_pin_header_2.54mm_smd_rl:10129380-902001BLF") (at 204.47 116.84 90) (unit 1)
     (in_bom yes) (on_board yes) (dnp no)
     (property "Reference" "P9" (at 200.66 115.57 90)
@@
       (effects (font (size 1.27 1.27)))
     )
-    (property "Footprint" "connector_smd_pinheader_2.54mm_rl:1x2_pinheader_2.54mm_vertical" (at 196.85 116.84 0)
+    (property "Footprint" "connector_pin_header_2.54mm_smd_rl:1x2_pin_header_2.54mm_vertical" (at 196.85 116.84 0)
       (effects (font (size 1.27 1.27)) hide)
     )
@@
     )
   )
-  (symbol (lib_id "connector_smd_pin_header_2.54mm_rl:10129380-902001BLF") (at 204.47 129.54 90) (unit 1)
+  (symbol (lib_id "connector_pin_header_2.54mm_smd_rl:10129380-902001BLF") (at 204.47 129.54 90) (unit 1)
     (in_bom yes) (on_board yes) (dnp no)
     (property "Reference" "P10" (at 200.66 128.27 90)
@@
       (effects (font (size 1.27 1.27)))
     )
-    (property "Footprint" "connector_smd_pinheader_2.54mm_rl:1x2_pinheader_2.54mm_vertical" (at 196.85 129.54 0)
+    (property "Footprint" "connector_pin_header_2.54mm_smd_rl:1x2_pin_header_2.54mm_vertical" (at 196.85 129.54 0)
       (effects (font (size 1.27 1.27)) hide)
     )
@@
     )
   )
-  (symbol (lib_id "connector_smd_pin_header_2.54mm_rl:10129380-902001BLF") (at 243.84 90.17 90) (unit 1)
+  (symbol (lib_id "connector_pin_header_2.54mm_smd_rl:10129380-902001BLF") (at 243.84 90.17 90) (unit 1)
     (in_bom yes) (on_board yes) (dnp no)
     (property "Reference" "P11" (at 240.03 87.63 90)
@@
       (effects (font (size 1.27 1.27)))
     )
-    (property "Footprint" "connector_smd_pinheader_2.54mm_rl:1x2_pinheader_2.54mm_vertical" (at 236.22 90.17 0)
+    (property "Footprint" "connector_pin_header_2.54mm_smd_rl:1x2_pin_header_2.54mm_vertical" (at 236.22 90.17 0)
       (effects (font (size 1.27 1.27)) hide)
     )
@@
     )
   )
-  (symbol (lib_id "connector_smd_pin_header_2.54mm_rl:10129380-902001BLF") (at 243.84 102.87 90) (unit 1)
+  (symbol (lib_id "connector_pin_header_2.54mm_smd_rl:10129380-902001BLF") (at 243.84 102.87 90) (unit 1)
     (in_bom yes) (on_board yes) (dnp no)
     (property "Reference" "P12" (at 238.76 100.33 90)
@@
       (effects (font (size 1.27 1.27)))
     )
-    (property "Footprint" "connector_smd_pinheader_2.54mm_rl:1x2_pinheader_2.54mm_vertical" (at 236.22 102.87 0)
+    (property "Footprint" "connector_pin_header_2.54mm_smd_rl:1x2_pin_header_2.54mm_vertical" (at 236.22 102.87 0)
       (effects (font (size 1.27 1.27)) hide)
     )
@@
     )
   )
-  (symbol (lib_id "connector_smd_pin_header_2.54mm_rl:10129380-902001BLF") (at 243.84 118.11 90) (unit 1)
+  (symbol (lib_id "connector_pin_header_2.54mm_smd_rl:10129380-902001BLF") (at 243.84 118.11 90) (unit 1)
     (in_bom yes) (on_board yes) (dnp no)
     (property "Reference" "P13" (at 240.03 115.57 90)
@@
       (effects (font (size 1.27 1.27)))
     )
-    (property "Footprint" "connector_smd_pinheader_2.54mm_rl:1x2_pinheader_2.54mm_vertical" (at 236.22 118.11 0)
+    (property "Footprint" "connector_pin_header_2.54mm_smd_rl:1x2_pin_header_2.54mm_vertical" (at 236.22 118.11 0)
       (effects (font (size 1.27 1.27)) hide)
     )
@@
     )
   )
-  (symbol (lib_id "connector_smd_pin_header_2.54mm_rl:10129380-902001BLF") (at 243.84 130.81 90) (unit 1)
+  (symbol (lib_id "connector_pin_header_2.54mm_smd_rl:10129380-902001BLF") (at 243.84 130.81 90) (unit 1)
     (in_bom yes) (on_board yes) (dnp no)
     (property "Reference" "P14" (at 240.03 128.27 90)
@@
       (effects (font (size 1.27 1.27)))
     )
-    (property "Footprint" "connector_smd_pinheader_2.54mm_rl:1x2_pinheader_2.54mm_vertical" (at 236.22 130.81 0)
+    (property "Footprint" "connector_pin_header_2.54mm_smd_rl:1x2_pin_header_2.54mm_vertical" (at 236.22 130.81 0)
       (effects (font (size 1.27 1.27)) hide)
     )
@@
     )
   )
-  (symbol (lib_id "connector_tht_pin_header_2.54mm_rl:DS1021-1-4SF11-B") (at 26.67 167.64 90) (unit 1)
+  (symbol (lib_id "connector_pin_header_2.54mm_tht_rl:DS1021-1-4SF11-B") (at 26.67 167.64 90) (unit 1)
     (in_bom yes) (on_board yes) (dnp no)
     (property "Reference" "P3" (at 26.67 161.29 90)
@@
       (effects (font (size 1.27 1.27)))
     )
-    (property "Footprint" "connector_tht_pinheader_2.54mm_rl:1x4_pinheader_2.54mm_vertical" (at 19.05 167.64 0)
+    (property "Footprint" "connector_pin_header_2.54mm_tht_rl:1x4_pin_header_2.54mm_vertical" (at 19.05 167.64 0)
       (effects (font (size 1.27 1.27)) hide)
     )
@@
     )
   )
-  (symbol (lib_id "connector_tht_pin_header_2.54mm_rl:DS1021-1-3SF11-B") (at 26.67 100.33 90) (unit 1)
+  (symbol (lib_id "connector_pin_header_2.54mm_tht_rl:DS1021-1-3SF11-B") (at 26.67 100.33 90) (unit 1)
     (in_bom yes) (on_board yes) (dnp no)
     (property "Reference" "P1" (at 26.67 93.98 90)
@@
       (effects (font (size 1.27 1.27)))
     )
-    (property "Footprint" "connector_tht_pinheader_2.54mm_rl:1x3_pinheader_2.54mm_vertical" (at 19.05 99.06 0)
-      (effects (font (size 1.27 1.27)) hide)
-    )
+    (property "Footprint" "connector_pin_header_2.54mm_tht_rl:1x3_pin_header_2.54mm_vertical" (at 19.05 99.06 0)
+      (effects (font (size 1.27 1.27)) hide)
+    )
