File: kicad-v7.0.9/wall-mounted-room-temperature sensor-wifi/wall-mounted-room-temperature-sensor-wifi.kicad_sch (KiCad schematic)
At the start: 61 parts, among them J1 PC-GK2.1, P1 2x3_MLW06A, P2 DS1023-1-9S21, Q1 DMG2307L, SW1 TVAF18BB, SW2 TVAF18BB, SW3 B3F-4150, SW4 B3F-4150, SW5 B3F-4150, U1 TPS79633KTTR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

Commit message: Change components form library. Adding of BOM.
Parts:
- P1: footprint connector_idc_rl:2x3_MLW06A -> connector_idc_tht_rl:2x3_MLW06A; symbol connector_idc_rl:2x3_MLW06A -> connector_idc_tht_rl:2x3_MLW06A
- P2: footprint connector_tht_pinsocket_2.54mm_rl:1x9_pinsocket_2.54mm_vertical_8.5mm -> connector_pin_socket_2.54mm_tht_rl:1x9_pin_socket_2.54mm_vertical_8.5mm; symbol connector_tht_pin_socket_2.54mm_rl:DS1023-1-9S21 -> connector_pin_socket_2.54mm_tht_rl:DS1023-1-9S21
Changed lines of the file:
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@@
     )
   )
-  (symbol (lib_id "connector_idc_rl:2x3_MLW06A") (at 190.5 252.73 0) (mirror x) (unit 1)
+  (symbol (lib_id "connector_idc_tht_rl:2x3_MLW06A") (at 190.5 252.73 0) (mirror x) (unit 1)
     (in_bom yes) (on_board yes) (dnp no)
     (property "Reference" "P1" (at 185.9534 252.1966 0)
@@
       (effects (font (size 1.27 1.27)))
     )
-    (property "Footprint" "connector_idc_rl:2x3_MLW06A" (at 190.5 269.24 0)
+    (property "Footprint" "connector_idc_tht_rl:2x3_MLW06A" (at 190.5 269.24 0)
       (effects (font (size 1.27 1.27)) hide)
     )
@@
     )
   )
-  (symbol (lib_id "connector_tht_pin_socket_2.54mm_rl:DS1023-1-9S21") (at 240.03 46.99 0) (mirror y) (unit 1)
+  (symbol (lib_id "connector_pin_socket_2.54mm_tht_rl:DS1023-1-9S21") (at 240.03 46.99 0) (mirror y) (unit 1)
     (in_bom yes) (on_board yes) (dnp no)
     (property "Reference" "P2" (at 239.9284 42.1132 0)
@@
       (effects (font (size 1.27 1.27)))
     )
-    (property "Footprint" "connector_tht_pinsocket_2.54mm_rl:1x9_pinsocket_2.54mm_vertical_8.5mm" (at 240.03 39.37 0)
-      (effects (font (size 1.27 1.27)) hide)
-    )
+    (property "Footprint" "connector_pin_socket_2.54mm_tht_rl:1x9_pin_socket_2.54mm_vertical_8.5mm" (at 240.03 39.37 0)
+      (effects (font (size 1.27 1.27)) hide)
+    )
