File: kicad-v7.0.9/zone-controller/differential-i2c-bus.kicad_sch (KiCad schematic)
At the start: 35 parts, among them J16 1x4_idc_lsa, J17 54601-908WPLF, J18 1x4_idc_lsa, P10 10129380-902001BLF, P11 10129380-902001BLF, P12 10129380-902001BLF, P13 10129380-902001BLF, P14 10129380-902001BLF, P15 10129380-902001BLF, P16 10129380-902001BLF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

Commit message: Change components form library. Adding of BOM.
Parts:
- J16, J18: footprint connector_rl:1x4_idc_lsa_connector_general -> connector_idc_lsa_tht_rl:1x4_idc_lsa_connector_general; symbol connector_rl:1x4_idc_lsa -> connector_idc_lsa_tht_rl:1x4_idc_lsa
- P10, P11, P12, P13, P14, P15, P16, P7, P8, P9: footprint connector_smd_pinheader_2.54mm_rl:1x2_pinheader_2.54mm_vertical -> connector_pin_header_2.54mm_smd_rl:1x2_pin_header_2.54mm_vertical; symbol connector_smd_pin_header_2.54mm_rl:10129380-902001BLF -> connector_pin_header_2.54mm_smd_rl:10129380-902001BLF
Changed lines of the file:
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@@
     )
   )
-  (symbol (lib_id "connector_smd_pin_header_2.54mm_rl:10129380-902001BLF") (at 120.65 83.82 90) (unit 1)
+  (symbol (lib_id "connector_pin_header_2.54mm_smd_rl:10129380-902001BLF") (at 120.65 83.82 90) (unit 1)
     (in_bom yes) (on_board yes) (dnp no)
     (property "Reference" "P7" (at 116.84 82.55 90)
@@
       (effects (font (size 1.27 1.27)))
     )
-    (property "Footprint" "connector_smd_pinheader_2.54mm_rl:1x2_pinheader_2.54mm_vertical" (at 113.03 83.82 0)
+    (property "Footprint" "connector_pin_header_2.54mm_smd_rl:1x2_pin_header_2.54mm_vertical" (at 113.03 83.82 0)
       (effects (font (size 1.27 1.27)) hide)
     )
@@
     )
   )
-  (symbol (lib_id "connector_smd_pin_header_2.54mm_rl:10129380-902001BLF") (at 133.35 83.82 90) (unit 1)
+  (symbol (lib_id "connector_pin_header_2.54mm_smd_rl:10129380-902001BLF") (at 133.35 83.82 90) (unit 1)
     (in_bom yes) (on_board yes) (dnp no)
     (property "Reference" "P8" (at 130.81 82.55 90)
@@
       (effects (font (size 1.27 1.27)))
     )
-    (property "Footprint" "connector_smd_pinheader_2.54mm_rl:1x2_pinheader_2.54mm_vertical" (at 125.73 83.82 0)
+    (property "Footprint" "connector_pin_header_2.54mm_smd_rl:1x2_pin_header_2.54mm_vertical" (at 125.73 83.82 0)
       (effects (font (size 1.27 1.27)) hide)
     )
@@
     )
   )
-  (symbol (lib_id "connector_rl:1x4_idc_lsa") (at 36.83 149.86 0) (unit 1)
+  (symbol (lib_id "connector_idc_lsa_tht_rl:1x4_idc_lsa") (at 36.83 149.86 0) (unit 1)
     (in_bom yes) (on_board yes) (dnp no)
     (property "Reference" "J16" (at 42.8752 150.7744 0)
@@
       (effects (font (size 1.27 1.27)) (justify left))
     )
-    (property "Footprint" "connector_rl:1x4_idc_lsa_connector_general" (at 35.56 149.86 90)
+    (property "Footprint" "connector_idc_lsa_tht_rl:1x4_idc_lsa_connector_general" (at 36.83 144.78 0)
       (effects (font (size 1.27 1.27)) hide)
     )
@@
     )
   )
-  (symbol (lib_id "connector_rl:1x4_idc_lsa") (at 60.96 149.86 0) (unit 1)
+  (symbol (lib_id "connector_idc_lsa_tht_rl:1x4_idc_lsa") (at 60.96 149.86 0) (unit 1)
     (in_bom yes) (on_board yes) (dnp no)
     (property "Reference" "J18" (at 67.0052 150.7744 0)
@@
       (effects (font (size 1.27 1.27)) (justify left))
     )
-    (property "Footprint" "connector_rl:1x4_idc_lsa_connector_general" (at 59.69 149.86 90)
+    (property "Footprint" "connector_idc_lsa_tht_rl:1x4_idc_lsa_connector_general" (at 60.96 144.78 0)
       (effects (font (size 1.27 1.27)) hide)
     )
@@
     )
   )
-  (symbol (lib_id "connector_smd_pin_header_2.54mm_rl:10129380-902001BLF") (at 209.55 57.15 90) (unit 1)
+  (symbol (lib_id "connector_pin_header_2.54mm_smd_rl:10129380-902001BLF") (at 209.55 57.15 90) (unit 1)
     (in_bom yes) (on_board yes) (dnp no)
     (property "Reference" "P9" (at 205.74 55.88 90)
@@
       (effects (font (size 1.27 1.27)))
     )
-    (property "Footprint" "connector_smd_pinheader_2.54mm_rl:1x2_pinheader_2.54mm_vertical" (at 201.93 57.15 0)
+    (property "Footprint" "connector_pin_header_2.54mm_smd_rl:1x2_pin_header_2.54mm_vertical" (at 201.93 57.15 0)
       (effects (font (size 1.27 1.27)) hide)
     )
@@
     )
   )
-  (symbol (lib_id "connector_smd_pin_header_2.54mm_rl:10129380-902001BLF") (at 209.55 95.25 90) (unit 1)
+  (symbol (lib_id "connector_pin_header_2.54mm_smd_rl:10129380-902001BLF") (at 209.55 95.25 90) (unit 1)
     (in_bom yes) (on_board yes) (dnp no)
     (property "Reference" "P12" (at 205.74 92.71 90)
@@
       (effects (font (size 1.27 1.27)))
     )
-    (property "Footprint" "connector_smd_pinheader_2.54mm_rl:1x2_pinheader_2.54mm_vertical" (at 201.93 95.25 0)
+    (property "Footprint" "connector_pin_header_2.54mm_smd_rl:1x2_pin_header_2.54mm_vertical" (at 201.93 95.25 0)
       (effects (font (size 1.27 1.27)) hide)
     )
@@
     )
   )
-  (symbol (lib_id "connector_smd_pin_header_2.54mm_rl:10129380-902001BLF") (at 209.55 68.58 90) (unit 1)
+  (symbol (lib_id "connector_pin_header_2.54mm_smd_rl:10129380-902001BLF") (at 209.55 68.58 90) (unit 1)
     (in_bom yes) (on_board yes) (dnp no)
     (property "Reference" "P10" (at 205.74 67.31 90)
@@
       (effects (font (size 1.27 1.27)))
     )
-    (property "Footprint" "connector_smd_pinheader_2.54mm_rl:1x2_pinheader_2.54mm_vertical" (at 201.93 68.58 0)
+    (property "Footprint" "connector_pin_header_2.54mm_smd_rl:1x2_pin_header_2.54mm_vertical" (at 201.93 68.58 0)
       (effects (font (size 1.27 1.27)) hide)
     )
@@
     )
   )
-  (symbol (lib_id "connector_smd_pin_header_2.54mm_rl:10129380-902001BLF") (at 209.55 83.82 90) (unit 1)
+  (symbol (lib_id "connector_pin_header_2.54mm_smd_rl:10129380-902001BLF") (at 209.55 83.82 90) (unit 1)
     (in_bom yes) (on_board yes) (dnp no)
     (property "Reference" "P11" (at 205.74 81.28 90)
@@
       (effects (font (size 1.27 1.27)))
     )
-    (property "Footprint" "connector_smd_pinheader_2.54mm_rl:1x2_pinheader_2.54mm_vertical" (at 201.93 83.82 0)
+    (property "Footprint" "connector_pin_header_2.54mm_smd_rl:1x2_pin_header_2.54mm_vertical" (at 201.93 83.82 0)
       (effects (font (size 1.27 1.27)) hide)
     )
@@
     )
   )
-  (symbol (lib_id "connector_smd_pin_header_2.54mm_rl:10129380-902001BLF") (at 257.81 58.42 90) (unit 1)
+  (symbol (lib_id "connector_pin_header_2.54mm_smd_rl:10129380-902001BLF") (at 257.81 58.42 90) (unit 1)
     (in_bom yes) (on_board yes) (dnp no)
     (property "Reference" "P13" (at 254 57.15 90)
@@
       (effects (font (size 1.27 1.27)))
     )
-    (property "Footprint" "connector_smd_pinheader_2.54mm_rl:1x2_pinheader_2.54mm_vertical" (at 250.19 58.42 0)
+    (property "Footprint" "connector_pin_header_2.54mm_smd_rl:1x2_pin_header_2.54mm_vertical" (at 250.19 58.42 0)
       (effects (font (size 1.27 1.27)) hide)
     )
@@
     )
   )
-  (symbol (lib_id "connector_smd_pin_header_2.54mm_rl:10129380-902001BLF") (at 257.81 96.52 90) (unit 1)
+  (symbol (lib_id "connector_pin_header_2.54mm_smd_rl:10129380-902001BLF") (at 257.81 96.52 90) (unit 1)
     (in_bom yes) (on_board yes) (dnp no)
     (property "Reference" "P16" (at 254 95.25 90)
@@
       (effects (font (size 1.27 1.27)))
     )
-    (property "Footprint" "connector_smd_pinheader_2.54mm_rl:1x2_pinheader_2.54mm_vertical" (at 250.19 96.52 0)
+    (property "Footprint" "connector_pin_header_2.54mm_smd_rl:1x2_pin_header_2.54mm_vertical" (at 250.19 96.52 0)
       (effects (font (size 1.27 1.27)) hide)
     )
@@
     )
   )
-  (symbol (lib_id "connector_smd_pin_header_2.54mm_rl:10129380-902001BLF") (at 257.81 69.85 90) (unit 1)
+  (symbol (lib_id "connector_pin_header_2.54mm_smd_rl:10129380-902001BLF") (at 257.81 69.85 90) (unit 1)
     (in_bom yes) (on_board yes) (dnp no)
     (property "Reference" "P14" (at 254 68.58 90)
@@
       (effects (font (size 1.27 1.27)))
     )
-    (property "Footprint" "connector_smd_pinheader_2.54mm_rl:1x2_pinheader_2.54mm_vertical" (at 250.19 69.85 0)
+    (property "Footprint" "connector_pin_header_2.54mm_smd_rl:1x2_pin_header_2.54mm_vertical" (at 250.19 69.85 0)
       (effects (font (size 1.27 1.27)) hide)
     )
@@
     )
   )
-  (symbol (lib_id "connector_smd_pin_header_2.54mm_rl:10129380-902001BLF") (at 257.81 85.09 90) (unit 1)
+  (symbol (lib_id "connector_pin_header_2.54mm_smd_rl:10129380-902001BLF") (at 257.81 85.09 90) (unit 1)
     (in_bom yes) (on_board yes) (dnp no)
     (property "Reference" "P15" (at 254 83.82 90)
@@
       (effects (font (size 1.27 1.27)))
     )
-    (property "Footprint" "connector_smd_pinheader_2.54mm_rl:1x2_pinheader_2.54mm_vertical" (at 250.19 85.09 0)
-      (effects (font (size 1.27 1.27)) hide)
-    )
+    (property "Footprint" "connector_pin_header_2.54mm_smd_rl:1x2_pin_header_2.54mm_vertical" (at 250.19 85.09 0)
+      (effects (font (size 1.27 1.27)) hide)
+    )
