File: kicad-v7.0.9/zone-controller/zone-controller.kicad_sch (KiCad schematic)
At the start: 61 parts, among them J15 EBBA-02-C-SS-BU, P1 95293-101A03LF, P2 95293-101A03LF, P3 95293-101A03LF, P4 95293-101A03LF, P5 95293-101A03LF, P6 95293-101A03LF, Q13 PMV213SN,215, Q14 PMV213SN,215, SW13 SMTS-102-2C2T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

Commit message: Change components form library. Adding of BOM.
Parts:
- P1, P2, P3, P4, P5, P6: footprint connector_smd_pinheader_2.54mm_rl:1x3_pinheader_2.54mm_vertical -> connector_pin_header_2.54mm_smd_rl:1x3_pin_header_2.54mm_vertical; symbol connector_smd_pin_header_2.54mm_rl:95293-101A03LF -> connector_pin_header_2.54mm_smd_rl:95293-101A03LF
Changed lines of the file:
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@@
       (effects (font (size 1.27 1.27)))
     )
-    (property "Footprint" "switch_tht_rl:SMTS-102-2C2T" (at 374.65 207.01 0)
-      (effects (font (size 1.27 1.27)) hide)
-    )
-    (property "Datasheet" "https://www.gme.cz/data/attachments/dsh.631-528.1.pdf" (at 374.65 207.01 0)
+    (property "Footprint" "switch_tht_rl:SMTS-102-2C2T" (at 361.95 208.28 0)
+      (effects (font (size 1.27 1.27)) hide)
+    )
+    (property "Datasheet" "https://www.gme.cz/data/attachments/dsh.631-528.1.pdf" (at 364.49 208.28 0)
       (effects (font (size 1.27 1.27)) hide)
     )
@@
     )
   )
-  (symbol (lib_id "connector_smd_pin_header_2.54mm_rl:95293-101A03LF") (at 290.83 43.18 90) (unit 1)
+  (symbol (lib_id "connector_pin_header_2.54mm_smd_rl:95293-101A03LF") (at 290.83 43.18 90) (unit 1)
     (in_bom yes) (on_board yes) (dnp no)
     (property "Reference" "P2" (at 290.83 38.1 90)
@@
       (effects (font (size 1.27 1.27)))
     )
-    (property "Footprint" "connector_smd_pinheader_2.54mm_rl:1x3_pinheader_2.54mm_vertical" (at 283.21 43.18 0)
+    (property "Footprint" "connector_pin_header_2.54mm_smd_rl:1x3_pin_header_2.54mm_vertical" (at 283.21 43.18 0)
       (effects (font (size 1.27 1.27)) hide)
     )
@@
     )
   )
-  (symbol (lib_id "connector_smd_pin_header_2.54mm_rl:95293-101A03LF") (at 308.61 43.18 90) (unit 1)
+  (symbol (lib_id "connector_pin_header_2.54mm_smd_rl:95293-101A03LF") (at 308.61 43.18 90) (unit 1)
     (in_bom yes) (on_board yes) (dnp no)
     (property "Reference" "P3" (at 308.61 38.1 90)
@@
       (effects (font (size 1.27 1.27)))
     )
-    (property "Footprint" "connector_smd_pinheader_2.54mm_rl:1x3_pinheader_2.54mm_vertical" (at 300.99 43.18 0)
+    (property "Footprint" "connector_pin_header_2.54mm_smd_rl:1x3_pin_header_2.54mm_vertical" (at 300.99 43.18 0)
       (effects (font (size 1.27 1.27)) hide)
     )
@@
     )
   )
-  (symbol (lib_id "connector_smd_pin_header_2.54mm_rl:95293-101A03LF") (at 326.39 43.18 90) (unit 1)
+  (symbol (lib_id "connector_pin_header_2.54mm_smd_rl:95293-101A03LF") (at 326.39 43.18 90) (unit 1)
     (in_bom yes) (on_board yes) (dnp no)
     (property "Reference" "P4" (at 326.39 38.1 90)
@@
       (effects (font (size 1.27 1.27)))
     )
-    (property "Footprint" "connector_smd_pinheader_2.54mm_rl:1x3_pinheader_2.54mm_vertical" (at 318.77 43.18 0)
+    (property "Footprint" "connector_pin_header_2.54mm_smd_rl:1x3_pin_header_2.54mm_vertical" (at 318.77 43.18 0)
       (effects (font (size 1.27 1.27)) hide)
     )
@@
     )
   )
-  (symbol (lib_id "connector_smd_pin_header_2.54mm_rl:95293-101A03LF") (at 344.17 43.18 90) (unit 1)
+  (symbol (lib_id "connector_pin_header_2.54mm_smd_rl:95293-101A03LF") (at 344.17 43.18 90) (unit 1)
     (in_bom yes) (on_board yes) (dnp no)
     (property "Reference" "P5" (at 344.17 38.1 90)
@@
       (effects (font (size 1.27 1.27)))
     )
-    (property "Footprint" "connector_smd_pinheader_2.54mm_rl:1x3_pinheader_2.54mm_vertical" (at 336.55 43.18 0)
+    (property "Footprint" "connector_pin_header_2.54mm_smd_rl:1x3_pin_header_2.54mm_vertical" (at 336.55 43.18 0)
       (effects (font (size 1.27 1.27)) hide)
     )
@@
     )
   )
-  (symbol (lib_id "connector_smd_pin_header_2.54mm_rl:95293-101A03LF") (at 361.95 43.18 90) (unit 1)
+  (symbol (lib_id "connector_pin_header_2.54mm_smd_rl:95293-101A03LF") (at 361.95 43.18 90) (unit 1)
     (in_bom yes) (on_board yes) (dnp no)
     (property "Reference" "P6" (at 361.95 38.1 90)
@@
       (effects (font (size 1.27 1.27)))
     )
-    (property "Footprint" "connector_smd_pinheader_2.54mm_rl:1x3_pinheader_2.54mm_vertical" (at 354.33 43.18 0)
+    (property "Footprint" "connector_pin_header_2.54mm_smd_rl:1x3_pin_header_2.54mm_vertical" (at 354.33 43.18 0)
       (effects (font (size 1.27 1.27)) hide)
     )
@@
     )
   )
-  (symbol (lib_id "connector_smd_pin_header_2.54mm_rl:95293-101A03LF") (at 273.05 43.18 90) (unit 1)
+  (symbol (lib_id "connector_pin_header_2.54mm_smd_rl:95293-101A03LF") (at 273.05 43.18 90) (unit 1)
     (in_bom yes) (on_board yes) (dnp no)
     (property "Reference" "P1" (at 273.05 38.1 90)
@@
       (effects (font (size 1.27 1.27)))
     )
-    (property "Footprint" "connector_smd_pinheader_2.54mm_rl:1x3_pinheader_2.54mm_vertical" (at 265.43 43.18 0)
-      (effects (font (size 1.27 1.27)) hide)
-    )
+    (property "Footprint" "connector_pin_header_2.54mm_smd_rl:1x3_pin_header_2.54mm_vertical" (at 265.43 43.18 0)
+      (effects (font (size 1.27 1.27)) hide)
+    )
